File: EAGLE/untitled.brd (EAGLE design)
At the start: 28 parts

Commit message: .
Parts:
- added N29, N30, N31, N32, N33, N34, N35, N36, N37, N38, N39, N40, N41, N42, N43, N44, N45, N46, N47, N48, N49, N50, N51, N52, N53, N54: IN-3, in3:IN-3
Connections:
- removed net N$10: N11.A
- removed net N$21: N10.A
Changed lines of the file:
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@@
 <board>
 <plain>
-<dimension x1="133" y1="41" x2="152" y2="-41" x3="-40" y3="0" layer="20" dtype="vertical"/>
-<dimension x1="-27" y1="-53" x2="27" y2="-54" x3="0" y3="50" layer="20" dtype="horizontal"/>
-<dimension x1="18" y1="-69" x2="38" y2="-72" x3="28" y3="77" layer="20" dtype="horizontal"/>
+<dimension x1="211" y1="41" x2="210" y2="-41" x3="-40" y3="0" layer="20" dtype="vertical"/>
+<dimension x1="-27" y1="-53" x2="27" y2="-54" x3="0" y3="46" layer="20" dtype="horizontal"/>
+<dimension x1="197" y1="-59" x2="143" y2="-60" x3="170" y3="47" layer="20" dtype="horizontal"/>
 <dimension x1="-57" y1="-26" x2="-51" y2="-41" x3="-98" y3="-33.5" layer="20" dtype="vertical"/>
-<dimension x1="108" y1="26" x2="107" y2="-26" x3="-76" y3="0" layer="20" dtype="vertical"/>
-<dimension x1="28" y1="-60" x2="82" y2="-59" x3="55" y3="47" layer="20" dtype="horizontal"/>
+<dimension x1="218" y1="12" x2="216" y2="26" x3="-76" y3="19" layer="20" dtype="vertical"/>
+<dimension x1="27" y1="50" x2="81" y2="-59" x3="54" y3="57" layer="20" dtype="horizontal"/>
+<dimension x1="89" y1="-58" x2="143" y2="51" x3="116" y3="57" layer="20" dtype="horizontal"/>
+<dimension x1="-27" y1="57" x2="197" y2="55" x3="85" y3="70" layer="20" dtype="horizontal"/>
 </plain>
 <attributes>
@@
 <element name="N27" library="in3" package="IN-3" value="IN-3" x="85" y="14"/>
 <element name="N28" library="in3" package="IN-3" value="IN-3" x="85" y="-14"/>
+<element name="N29" library="in3" package="IN-3" value="IN-3" x="102" y="28" rot="R135"/>
+<element name="N30" library="in3" package="IN-3" value="IN-3" x="116" y="28" rot="R135"/>
+<element name="N31" library="in3" package="IN-3" value="IN-3" x="130" y="28" rot="R135"/>
+<element name="N32" library="in3" package="IN-3" value="IN-3" x="130" y="14" rot="R135"/>
+<element name="N33" library="in3" package="IN-3" value="IN-3" x="130" y="0" rot="R135"/>
+<element name="N34" library="in3" package="IN-3" value="IN-3" x="130" y="-14" rot="R135"/>
+<element name="N35" library="in3" package="IN-3" value="IN-3" x="130" y="-28" rot="R315"/>
+<element name="N36" library="in3" package="IN-3" value="IN-3" x="116" y="-28" rot="R315"/>
+<element name="N37" library="in3" package="IN-3" value="IN-3" x="102" y="-28" rot="R315"/>
+<element name="N38" library="in3" package="IN-3" value="IN-3" x="102" y="-14" rot="R315"/>
+<element name="N39" library="in3" package="IN-3" value="IN-3" x="102" y="0" rot="R315"/>
+<element name="N40" library="in3" package="IN-3" value="IN-3" x="102" y="14" rot="R315"/>
+<element name="N41" library="in3" package="IN-3" value="IN-3" x="116" y="0"/>
+<element name="N42" library="in3" package="IN-3" value="IN-3" x="156" y="28" rot="R225"/>
+<element name="N43" library="in3" package="IN-3" value="IN-3" x="170" y="28" rot="R225"/>
+<element name="N44" library="in3" package="IN-3" value="IN-3" x="184" y="28" rot="R225"/>
+<element name="N45" library="in3" package="IN-3" value="IN-3" x="184" y="14" rot="R45"/>
+<element name="N46" library="in3" package="IN-3" value="IN-3" x="184" y="0" rot="R45"/>
+<element name="N47" library="in3" package="IN-3" value="IN-3" x="184" y="-14" rot="R45"/>
+<element name="N48" library="in3" package="IN-3" value="IN-3" x="184" y="-28" rot="R45"/>
+<element name="N49" library="in3" package="IN-3" value="IN-3" x="170" y="-28" rot="R45"/>
+<element name="N50" library="in3" package="IN-3" value="IN-3" x="156" y="-28" rot="R45"/>
+<element name="N51" library="in3" package="IN-3" value="IN-3" x="156" y="-14" rot="R225"/>
+<element name="N52" library="in3" package="IN-3" value="IN-3" x="156" y="0" rot="R225"/>
+<element name="N53" library="in3" package="IN-3" value="IN-3" x="156" y="14" rot="R225"/>
+<element name="N54" library="in3" package="IN-3" value="IN-3" x="170" y="0"/>
 </elements>
 <signals>
-<signal name="N$10">
-<contactref element="N11" pad="A"/>
-</signal>
-<signal name="N$21">
-<contactref element="N10" pad="A"/>
-</signal>
 </signals>
 </board>

Commit message: first commit
Parts:
- added DD1: MEGA8-AI, atmel:TQFP32-08
- added IC1, IC3: 74HC595D, 74xx-eu:SO16
Connections:
- new net AVCC: DD1.18
- new net GND: DD1.21, DD1.3, DD1.5, IC1.8, IC3.8
- new net VCC: DD1.4, DD1.6, IC1.16, IC3.16
Changed lines of the file:
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@@
 <layer number="25" name="tNames" color="7" fill="1" visible="yes" active="yes"/>
 <layer number="26" name="bNames" color="7" fill="1" visible="yes" active="yes"/>
-<layer number="27" name="tValues" color="7" fill="1" visible="yes" active="yes"/>
-<layer number="28" name="bValues" color="7" fill="1" visible="yes" active="yes"/>
+<layer number="27" name="tValues" color="7" fill="1" visible="no" active="yes"/>
+<layer number="28" name="bValues" color="7" fill="1" visible="no" active="yes"/>
 <layer number="29" name="tStop" color="7" fill="3" visible="no" active="yes"/>
 <layer number="30" name="bStop" color="7" fill="6" visible="no" active="yes"/>
@@
 <layer number="48" name="Document" color="7" fill="1" visible="yes" active="yes"/>
 <layer number="49" name="Reference" color="7" fill="1" visible="yes" active="yes"/>
-<layer number="51" name="tDocu" color="14" fill="1" visible="yes" active="yes"/>
+<layer number="51" name="tDocu" color="15" fill="1" visible="yes" active="yes"/>
 <layer number="52" name="bDocu" color="7" fill="1" visible="yes" active="yes"/>
 <layer number="91" name="Nets" color="2" fill="1" visible="no" active="no"/>
@@
 <dimension x1="211" y1="41" x2="210" y2="-41" x3="-40" y3="0" layer="20" dtype="vertical"/>
 <dimension x1="-27" y1="-53" x2="27" y2="-54" x3="0" y3="46" layer="20" dtype="horizontal"/>
-<dimension x1="197" y1="-59" x2="143" y2="-60" x3="170" y3="47" layer="20" dtype="horizontal"/>
-<dimension x1="-57" y1="-26" x2="-51" y2="-41" x3="-98" y3="-33.5" layer="20" dtype="vertical"/>
-<dimension x1="218" y1="12" x2="216" y2="26" x3="-76" y3="19" layer="20" dtype="vertical"/>
-<dimension x1="27" y1="50" x2="81" y2="-59" x3="54" y3="57" layer="20" dtype="horizontal"/>
-<dimension x1="89" y1="-58" x2="143" y2="51" x3="116" y3="57" layer="20" dtype="horizontal"/>
+<dimension x1="197" y1="-59" x2="143" y2="-60" x3="170" y3="46" layer="20" dtype="horizontal"/>
+<dimension x1="27" y1="50" x2="81" y2="-59" x3="54" y3="55" layer="20" dtype="horizontal"/>
+<dimension x1="89" y1="-58" x2="143" y2="51" x3="116" y3="55" layer="20" dtype="horizontal"/>
 <dimension x1="-27" y1="57" x2="197" y2="55" x3="85" y3="70" layer="20" dtype="horizontal"/>
+<circle x="143" y="-31" radius="10" width="0.4064" layer="21"/>
 </plain>
 <attributes>
@@
 </class>
 </classes>
-<designrules name="default">
-<description language="de">&lt;b&gt;EAGLE Design Rules&lt;/b&gt;
+<designrules name="DesignRules">
+<description language="de">
+&lt;b&gt;EAGLE Design Rules&lt;/b&gt;
+</description>
+<description language="en">
+&lt;b&gt;EAGLE Design Rules&lt;/b&gt;
 &lt;p&gt;
-Die Standard-Design-Rules sind so gewählt, dass sie für
-die meisten Anwendungen passen. Sollte ihre Platine
-besondere Anforderungen haben, treffen Sie die erforderlichen
-Einstellungen hier und speichern die Design Rules unter
-einem neuen Namen ab.</description>
-<description language="en">&lt;b&gt;EAGLE Design Rules&lt;/b&gt;
-&lt;p&gt;
-The default Design Rules have been set to cover
-a wide range of applications. Your particular design
-may have different requirements, so please make the
-necessary adjustments and save your customized
-design rules under a new name.</description>
+</description>
 <param name="layerSetup" value="(1*16)"/>
 <param name="mtCopper" value="0.035mm 0.035mm 0.035mm 0.035mm 0.035mm 0.035mm 0.035mm 0.035mm 0.035mm 0.035mm 0.035mm 0.035mm 0.035mm 0.035mm 0.035mm 0.035mm"/>
 <param name="mtIsolate" value="1.5mm 0.15mm 0.2mm 0.15mm 0.2mm 0.15mm 0.2mm 0.15mm 0.2mm 0.15mm 0.2mm 0.15mm 0.2mm 0.15mm 0.2mm"/>
-<param name="mdWireWire" value="8mil"/>
-<param name="mdWirePad" value="8mil"/>
-<param name="mdWireVia" value="8mil"/>
+<param name="mdWireWire" value="0.2mm"/>
+<param name="mdWirePad" value="0.2mm"/>
+<param name="mdWireVia" value="0.2mm"/>
 <param name="mdPadPad" value="8mil"/>
 <param name="mdPadVia" value="8mil"/>
@@
 <param name="mdViaViaSameLayer" value="8mil"/>
 <param name="mnLayersViaInSmd" value="2"/>
-<param name="mdCopperDimension" value="40mil"/>
+<param name="mdCopperDimension" value="10mil"/>
 <param name="mdDrill" value="8mil"/>
 <param name="mdSmdStop" value="0mil"/>
-<param name="msWidth" value="10mil"/>
+<param name="msWidth" value="8mil"/>
 <param name="msDrill" value="24mil"/>
 <param name="msMicroVia" value="9.99mm"/>
 <param name="msBlindViaRatio" value="0.5"/>
-<param name="rvPadTop" value="0.25"/>
-<param name="rvPadInner" value="0.25"/>
-<param name="rvPadBottom" value="0.25"/>
+<param name="rvPadTop" value="0.2"/>
+<param name="rvPadInner" value="0.3"/>
+<param name="rvPadBottom" value="0.2"/>
 <param name="rvViaOuter" value="0.25"/>
 <param name="rvViaInner" value="0.25"/>
 <param name="rvMicroViaOuter" value="0.25"/>
 <param name="rvMicroViaInner" value="0.25"/>
-<param name="rlMinPadTop" value="10mil"/>
-<param name="rlMaxPadTop" value="20mil"/>
+<param name="rlMinPadTop" value="0.55mm"/>
+<param name="rlMaxPadTop" value="1mm"/>
 <param name="rlMinPadInner" value="10mil"/>
 <param name="rlMaxPadInner" value="20mil"/>
-<param name="rlMinPadBottom" value="10mil"/>
-<param name="rlMaxPadBottom" value="20mil"/>
+<param name="rlMinPadBottom" value="0.55mm"/>
+<param name="rlMaxPadBottom" value="1mm"/>
 <param name="rlMinViaOuter" value="8mil"/>
 <param name="rlMaxViaOuter" value="20mil"/>
@@
 <element name="N53" library="in3" package="IN-3" value="IN-3" x="156" y="14" rot="R225"/>
 <element name="N54" library="in3" package="IN-3" value="IN-3" x="170" y="0"/>
+<element name="IC1" library="74xx-eu" package="SO16" value="74HC595D" x="185" y="-27" rot="MR270"/>
+<element name="DD1" library="atmel" package="TQFP32-08" value="MEGA8-AI" x="116" y="16" rot="MR270">
+<attribute name="OC_NEWARK" value="73M8863" x="116" y="16" size="1.778" layer="28" rot="MR270" display="off"/>
+<attribute name="MPN" value="ATMEGA8-16AU" x="116" y="16" size="1.778" layer="28" rot="MR270" display="off"/>
+<attribute name="MF" value="" x="116" y="16" size="1.778" layer="28" rot="MR270" display="off"/>
+<attribute name="OC_FARNELL" value="9171371" x="116" y="16" size="1.778" layer="28" rot="MR270" display="off"/>
+</element>
+<element name="IC3" library="74xx-eu" package="SO16" value="74HC595D" x="159" y="23" rot="MR270"/>
 </elements>
 <signals>
+<signal name="GND">
+<contactref element="IC1" pad="8"/>
+<contactref element="DD1" pad="3"/>
+<contactref element="DD1" pad="5"/>
+<contactref element="DD1" pad="21"/>
+<contactref element="IC3" pad="8"/>
+<wire x1="116.4" y1="20.2926" x2="162.0734" y2="18.555" width="0" layer="19" extent="16-16"/>
+<wire x1="114.8" y1="20.2926" x2="116.4" y2="20.2926" width="0" layer="19" extent="16-16"/>
+<wire x1="115.6" y1="11.7074" x2="116.4" y2="20.2926" width="0" layer="19" extent="16-16"/>
+<wire x1="188.0734" y1="-31.445" x2="162.0734" y2="18.555" width="0" layer="19" extent="16-16"/>
+</signal>
+<signal name="VCC">
+<contactref element="IC1" pad="16"/>
+<contactref element="DD1" pad="4"/>
+<contactref element="DD1" pad="6"/>
+<contactref element="IC3" pad="16"/>
+<wire x1="117.2" y1="20.2926" x2="155.9266" y2="27.445" width="0" layer="19" extent="16-16"/>
+<wire x1="115.6" y1="20.2926" x2="117.2" y2="20.2926" width="0" layer="19" extent="16-16"/>
+<wire x1="181.9266" y1="-22.555" x2="155.9266" y2="27.445" width="0" layer="19" extent="16-16"/>
+</signal>
+<signal name="AVCC">
+<contactref element="DD1" pad="18"/>
+</signal>
 </signals>
 </board>

Commit message: .
Parts:
- moved IC3 72.1 mm to (162.0, -49.0)
- moved DD1 64.0 mm to (118.0, -48.0)
- moved IC1 25.3 mm to (181.0, -52.0)
Changed lines of the file:
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@@
 <dimension x1="89" y1="-58" x2="143" y2="51" x3="116" y3="55" layer="20" dtype="horizontal"/>
 <dimension x1="-27" y1="57" x2="197" y2="55" x3="85" y3="70" layer="20" dtype="horizontal"/>
-<circle x="143" y="-31" radius="10" width="0.4064" layer="21"/>
+<circle x="139" y="-55" radius="10" width="0.4064" layer="21"/>
 </plain>
 <attributes>
@@
 <element name="N53" library="in3" package="IN-3" value="IN-3" x="156" y="14" rot="R225"/>
 <element name="N54" library="in3" package="IN-3" value="IN-3" x="170" y="0"/>
-<element name="IC1" library="74xx-eu" package="SO16" value="74HC595D" x="185" y="-27" rot="MR270"/>
-<element name="DD1" library="atmel" package="TQFP32-08" value="MEGA8-AI" x="116" y="16" rot="MR270">
-<attribute name="OC_NEWARK" value="73M8863" x="116" y="16" size="1.778" layer="28" rot="MR270" display="off"/>
-<attribute name="MPN" value="ATMEGA8-16AU" x="116" y="16" size="1.778" layer="28" rot="MR270" display="off"/>
-<attribute name="MF" value="" x="116" y="16" size="1.778" layer="28" rot="MR270" display="off"/>
-<attribute name="OC_FARNELL" value="9171371" x="116" y="16" size="1.778" layer="28" rot="MR270" display="off"/>
+<element name="IC1" library="74xx-eu" package="SO16" value="74HC595D" x="181" y="-52" rot="MR270"/>
+<element name="DD1" library="atmel" package="TQFP32-08" value="MEGA8-AI" x="118" y="-48" rot="MR270">
+<attribute name="OC_NEWARK" value="73M8863" x="118" y="-48" size="1.778" layer="28" rot="MR270" display="off"/>
+<attribute name="MPN" value="ATMEGA8-16AU" x="118" y="-48" size="1.778" layer="28" rot="MR270" display="off"/>
+<attribute name="MF" value="" x="118" y="-48" size="1.778" layer="28" rot="MR270" display="off"/>
+<attribute name="OC_FARNELL" value="9171371" x="118" y="-48" size="1.778" layer="28" rot="MR270" display="off"/>
 </element>
-<element name="IC3" library="74xx-eu" package="SO16" value="74HC595D" x="159" y="23" rot="MR270"/>
+<element name="IC3" library="74xx-eu" package="SO16" value="74HC595D" x="162" y="-49" rot="MR270"/>
 </elements>
 <signals>
@@
 <contactref element="DD1" pad="21"/>
 <contactref element="IC3" pad="8"/>
-<wire x1="116.4" y1="20.2926" x2="162.0734" y2="18.555" width="0" layer="19" extent="16-16"/>
-<wire x1="114.8" y1="20.2926" x2="116.4" y2="20.2926" width="0" layer="19" extent="16-16"/>
-<wire x1="115.6" y1="11.7074" x2="116.4" y2="20.2926" width="0" layer="19" extent="16-16"/>
-<wire x1="188.0734" y1="-31.445" x2="162.0734" y2="18.555" width="0" layer="19" extent="16-16"/>
+<wire x1="118.4" y1="-43.7074" x2="165.0734" y2="-53.445" width="0" layer="19" extent="16-16"/>
+<wire x1="116.8" y1="-43.7074" x2="118.4" y2="-43.7074" width="0" layer="19" extent="16-16"/>
+<wire x1="117.6" y1="-52.2926" x2="118.4" y2="-43.7074" width="0" layer="19" extent="16-16"/>
+<wire x1="184.0734" y1="-56.445" x2="165.0734" y2="-53.445" width="0" layer="19" extent="16-16"/>
 </signal>
 <signal name="VCC">
@@
 <contactref element="DD1" pad="6"/>
 <contactref element="IC3" pad="16"/>
-<wire x1="117.2" y1="20.2926" x2="155.9266" y2="27.445" width="0" layer="19" extent="16-16"/>
-<wire x1="115.6" y1="20.2926" x2="117.2" y2="20.2926" width="0" layer="19" extent="16-16"/>
-<wire x1="181.9266" y1="-22.555" x2="155.9266" y2="27.445" width="0" layer="19" extent="16-16"/>
+<wire x1="119.2" y1="-43.7074" x2="158.9266" y2="-44.555" width="0" layer="19" extent="16-16"/>
+<wire x1="117.6" y1="-43.7074" x2="119.2" y2="-43.7074" width="0" layer="19" extent="16-16"/>
+<wire x1="177.9266" y1="-47.555" x2="158.9266" y2="-44.555" width="0" layer="19" extent="16-16"/>
 </signal>
 <signal name="AVCC">
