File: EAGLE/in3watch.sch (EAGLE design)
At the start: 274 parts, among them IC1 74HC595D, IC2 74HC595D, IC3 74HC595D, IC4 74HC595D, IC5 74HC595D, IC6 74HC595D, IC7 74HC595D

Commit message: .
Parts:
- added ISP: (no value), con-lstb:MA03-2
- added Q1: (no value), crystal:CRYSTALHC49U70
Connections:
- new net MISO: DD2.PB4(MISO), ISP.1
- new net MOSI: DD2.PB3(MOSI/OC2), ISP.4
- new net N$112: DD2.PB6(XTAL1/TOSC1), Q1.2
- new net RESET: DD2.PC6(/RESET), ISP.5
- new net SCK: DD2.PB5(SCK), ISP.3
- net +5V: now also DD2.VCC@1, DD2.VCC@2, ISP.2
- net GND: now also ISP.6
- net N$72: now also DD2.PB7(XTAL2/TOSC2), Q1.1; no longer DD2.VCC@1, DD2.VCC@2

Commit message: 2
Parts:
- added C3, C4: (no value), rcl:C-EUC0805
- added Z1: 32768, zq:FC-12M
- DD2: value MEGA8-AI -> MEGA328P
Connections:
- net N$31 renamed VBAT
- net N$73 renamed SEQ
- net N$76 renamed SDA
- net N$77 renamed SCL
- new net N$31: DD1.X2, Z1.1
- net +5V: now also DD1.VCC
- net GND: now also C3.1, C4.1
- net N$112: now also C3.2
- net N$33: now also Z1.2; no longer DD1.X2
- net N$72: now also C4.2
Other:
- note added: "VT MMBTA42LT1G RB RC VZ 5V6"
- note removed: "MMBTA42LT1G"

Commit message: .
Parts:
- removed G1: CR2032H, battery:CR2032H
- added BT1: (no value), SparkFun-Batteries:BATTERY-20MM_PTH
Connections:
- net GND: now also BT1.-; no longer G1.-
- net VBAT: now also BT1.+; no longer G1.+

Commit message: .
Parts:
- added C5, C6: (no value), rcl:C-EUC0805
- added J1, J2: (no value), rcl:R-EU_R1206
- added R105, R109: 10k, rcl:R-EU_R1206W
- added R106, R107, R108: 10k, rcl:R-EU_R0805
- BT1: value (none) -> 2032 3v
- DD2: value MEGA328P -> ATMEGA328P
Connections:
- new net +5VISP: ISP.2, J1.1, R105.2
- new net N$73: R105.1, R109.2
- new net N$76: C3.1, C4.1, J2.2
- net +5V: now also C5.1, C6.1, J1.2, R106.2, R107.2, R108.2; no longer ISP.2
- net GND: now also C5.2, C6.2, J2.1; no longer C3.1, C4.1
- net RESET: now also R109.1
- net SCL: now also R108.1
- net SDA: now also R107.1
- net SEQ: now also R106.1
Other:
- moved on the sheet: C3, C4, ISP, Q1

Commit message: .
Parts:
- added J3: J5MM, in3wlbr:J5MM
- R19: device rcl:R-EU_R0805 -> rcl:R-EU_R1206W
Connections:
- net GND: now also J3.1, J3.2
Changed lines of the file:
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@@
 <part name="VD9" library="diode" deviceset="ZENER-DIODE" device="SOD80C"/>
 <part name="VT10" library="transistor-npn" deviceset="BC849*" device="SMD" value=""/>
-<part name="R19" library="rcl" deviceset="R-EU_" device="R0805"/>
+<part name="R19" library="rcl" deviceset="R-EU_" device="R1206W"/>
 <part name="R20" library="rcl" deviceset="R-EU_" device="0207/12"/>
 <part name="GND10" library="supply1" deviceset="GND" device=""/>
@@
 <part name="R105" library="rcl" deviceset="R-EU_" device="R1206W" value="10k"/>
 <part name="R109" library="rcl" deviceset="R-EU_" device="R1206W" value="10k"/>
+<part name="J3" library="in3wlbr" deviceset="J" device="5MM"/>
 </parts>
 <sheets>
@@
 <instance part="DD2" gate="G$1" x="91.44" y="68.58" rot="MR180"/>
 <instance part="DD1" gate="G$1" x="106.68" y="134.62"/>
-<instance part="GND36" gate="1" x="93.98" y="121.92"/>
+<instance part="GND36" gate="1" x="93.98" y="114.3"/>
 <instance part="GND37" gate="1" x="66.04" y="38.1" rot="MR0"/>
 <instance part="ISP" gate="1" x="20.32" y="83.82" smashed="yes" rot="R180">
@@
 <instance part="R105" gate="G$1" x="50.8" y="73.66" rot="R90"/>
 <instance part="R109" gate="G$1" x="50.8" y="53.34" rot="R90"/>
+<instance part="J3" gate="1" x="86.36" y="124.46"/>
 </instances>
 <busses>
@@
 <wire x1="93.98" y1="127" x2="96.52" y2="127" width="0.1524" layer="91"/>
 <pinref part="GND36" gate="1" pin="GND"/>
+<wire x1="93.98" y1="116.84" x2="93.98" y2="119.38" width="0.1524" layer="91"/>
+<pinref part="J3" gate="1" pin="2"/>
+<wire x1="93.98" y1="119.38" x2="93.98" y2="124.46" width="0.1524" layer="91"/>
 <wire x1="93.98" y1="124.46" x2="93.98" y2="127" width="0.1524" layer="91"/>
+<wire x1="91.44" y1="124.46" x2="93.98" y2="124.46" width="0.1524" layer="91"/>
+<wire x1="93.98" y1="119.38" x2="78.74" y2="119.38" width="0.1524" layer="91"/>
+<wire x1="78.74" y1="119.38" x2="78.74" y2="124.46" width="0.1524" layer="91"/>
+<pinref part="J3" gate="1" pin="1"/>
+<wire x1="78.74" y1="124.46" x2="81.28" y2="124.46" width="0.1524" layer="91"/>
+<junction x="93.98" y="119.38"/>
+<junction x="93.98" y="124.46"/>
 </segment>
 <segment>
@@
 <wire x1="50.8" y1="43.18" x2="38.1" y2="43.18" width="0.1524" layer="91"/>
 <wire x1="50.8" y1="48.26" x2="50.8" y2="43.18" width="0.1524" layer="91"/>
-</segment>
-</net>
+<junction x="50.8" y="43.18"/>
+</segment>
+</net>

Commit message: .
Parts:
- removed DD1: DS1307, ds1307_pcf8583:DS1307
- added C7: (no value), rcl:C-EUC0805
- added C8: (no value), rcl:C-EUC3225
- added DD1A: (no value), DS3231_industrialberry:DS3231SOIC-16W
- added DD1B: DS1307, ds1307_pcf8583:DS1307
- added J4, J5: (no value), rcl:R-EU_R1206W
- added R110, R113: 10k, rcl:R-EU_R0805
- added SJ1: (no value), jumper:SJ
Connections:
- removed net MISO: DD2.PB4(MISO), ISP.1
- removed net MOSI: DD2.PB3(MOSI/OC2), ISP.4
- removed net RCLOCK: IC1A.SCK, IC2A.SCK, IC3A.SCK, IC4A.SCK, IC5A.SCK, IC6A.SCK, IC7A.SCK
- removed net RDATA: IC1A.SER
- removed net RLATCH: IC1A.RCK, IC2A.RCK, IC3A.RCK, IC4A.RCK, IC5A.RCK, IC6A.RCK, IC7A.RCK
- new net N$114: DD1A.32KHZ, R110.1
- new net N$115: DD1A.!RST, R113.1
- new net RCLOCK_MISO_D12: DD2.PB4(MISO), IC1A.SCK, IC2A.SCK, IC3A.SCK, IC4A.SCK, IC5A.SCK, IC6A.SCK, IC7A.SCK, ISP.1
- new net RDATA_MOSI_D11: DD2.PB3(MOSI/OC2), IC1A.SER, ISP.4
- new net RLATCH_D10: DD2.PB2(SS/OC1B), IC1A.RCK, IC2A.RCK, IC3A.RCK, IC4A.RCK, IC5A.RCK, IC6A.RCK, IC7A.RCK
- new net SCL_J: DD1A.SCL, J4.1
- new net SEQ_J: DD1A.!INT, J5.2
- net +5V: now also C7.1, DD1A.VCC, DD1B.VCC, R110.2, R113.2; no longer DD1.VCC
- net GND: now also C7.2, C8.2, DD1A.GND, DD1A.NC@1, DD1A.NC@2, DD1A.NC@3, DD1A.NC@4, DD1A.NC@5, DD1A.NC@6, DD1A.NC@7, DD1A.NC@8, DD1B.GND, SJ1.1, SJ1.2; no longer DD1.GND
- net N$31: now also DD1B.X2; no longer DD1.X2
- net N$33: now also DD1B.X1; no longer DD1.X1
- net SCL: now also DD1B.SCL, J4.2; no longer DD1.SCL
- net SDA: now also DD1A.SDA, DD1B.SDA; no longer DD1.SDA
- net SEQ: now also DD1B.SQW, J5.1; no longer DD1.SQW
- net VBAT: now also C8.1, DD1A.VBAT, DD1B.VBAT; no longer DD1.VBAT

Commit message: .
Parts:
- R35: device rcl:R-EU_R0805 -> rcl:R-EU_M1206
- R37: device rcl:R-EU_R0805 -> rcl:R-EU_0204/7
- R39: device rcl:R-EU_R0805 -> rcl:R-EU_R1206W
Changed lines of the file:
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@@
 <grid distance="100" unitdist="mil" unit="mil" style="lines" multiple="1" display="yes" altdistance="0.01" altunitdist="inch" altunit="inch"/>
 <layers>
-<layer number="1" name="Top" color="4" fill="1" visible="no" active="no"/>
-<layer number="2" name="Route2" color="1" fill="3" visible="no" active="no"/>
-<layer number="3" name="Route3" color="4" fill="3" visible="no" active="no"/>
-<layer number="4" name="Route4" color="1" fill="4" visible="no" active="no"/>
-<layer number="5" name="Route5" color="4" fill="4" visible="no" active="no"/>
-<layer number="6" name="Route6" color="1" fill="8" visible="no" active="no"/>
-<layer number="7" name="Route7" color="4" fill="8" visible="no" active="no"/>
-<layer number="8" name="Route8" color="1" fill="2" visible="no" active="no"/>
-<layer number="9" name="Route9" color="4" fill="2" visible="no" active="no"/>
-<layer number="10" name="Route10" color="1" fill="7" visible="no" active="no"/>
-<layer number="11" name="Route11" color="4" fill="7" visible="no" active="no"/>
-<layer number="12" name="Route12" color="1" fill="5" visible="no" active="no"/>
-<layer number="13" name="Route13" color="4" fill="5" visible="no" active="no"/>
-<layer number="14" name="Route14" color="1" fill="6" visible="no" active="no"/>
-<layer number="15" name="Route15" color="4" fill="6" visible="no" active="no"/>
-<layer number="16" name="Bottom" color="1" fill="1" visible="no" active="no"/>
-<layer number="17" name="Pads" color="2" fill="1" visible="no" active="no"/>
-<layer number="18" name="Vias" color="2" fill="1" visible="no" active="no"/>
-<layer number="19" name="Unrouted" color="6" fill="1" visible="no" active="no"/>
-<layer number="20" name="Dimension" color="15" fill="1" visible="no" active="no"/>
-<layer number="21" name="tPlace" color="7" fill="1" visible="no" active="no"/>
-<layer number="22" name="bPlace" color="7" fill="1" visible="no" active="no"/>
-<layer number="23" name="tOrigins" color="15" fill="1" visible="no" active="no"/>
-<layer number="24" name="bOrigins" color="15" fill="1" visible="no" active="no"/>
-<layer number="25" name="tNames" color="7" fill="1" visible="no" active="no"/>
-<layer number="26" name="bNames" color="7" fill="1" visible="no" active="no"/>
-<layer number="27" name="tValues" color="7" fill="1" visible="no" active="no"/>
-<layer number="28" name="bValues" color="7" fill="1" visible="no" active="no"/>
+<layer number="1" name="Top" color="4" fill="1" visible="yes" active="no"/>
+<layer number="2" name="Route2" color="1" fill="3" visible="yes" active="no"/>
+<layer number="3" name="Route3" color="4" fill="3" visible="yes" active="no"/>
+<layer number="4" name="Route4" color="1" fill="4" visible="yes" active="no"/>
+<layer number="5" name="Route5" color="4" fill="4" visible="yes" active="no"/>
+<layer number="6" name="Route6" color="1" fill="8" visible="yes" active="no"/>
+<layer number="7" name="Route7" color="4" fill="8" visible="yes" active="no"/>
+<layer number="8" name="Route8" color="1" fill="2" visible="yes" active="no"/>
+<layer number="9" name="Route9" color="4" fill="2" visible="yes" active="no"/>
+<layer number="10" name="Route10" color="1" fill="7" visible="yes" active="no"/>
+<layer number="11" name="Route11" color="4" fill="7" visible="yes" active="no"/>
+<layer number="12" name="Route12" color="1" fill="5" visible="yes" active="no"/>
+<layer number="13" name="Route13" color="4" fill="5" visible="yes" active="no"/>
+<layer number="14" name="Route14" color="1" fill="6" visible="yes" active="no"/>
+<layer number="15" name="Route15" color="4" fill="6" visible="yes" active="no"/>
+<layer number="16" name="Bottom" color="1" fill="1" visible="yes" active="no"/>
+<layer number="17" name="Pads" color="2" fill="1" visible="yes" active="no"/>
+<layer number="18" name="Vias" color="2" fill="1" visible="yes" active="no"/>
+<layer number="19" name="Unrouted" color="6" fill="1" visible="yes" active="no"/>
+<layer number="20" name="Dimension" color="15" fill="1" visible="yes" active="no"/>
+<layer number="21" name="tPlace" color="7" fill="1" visible="yes" active="no"/>
+<layer number="22" name="bPlace" color="7" fill="1" visible="yes" active="no"/>
+<layer number="23" name="tOrigins" color="15" fill="1" visible="yes" active="no"/>
+<layer number="24" name="bOrigins" color="15" fill="1" visible="yes" active="no"/>
+<layer number="25" name="tNames" color="7" fill="1" visible="yes" active="no"/>
+<layer number="26" name="bNames" color="7" fill="1" visible="yes" active="no"/>
+<layer number="27" name="tValues" color="7" fill="1" visible="yes" active="no"/>
+<layer number="28" name="bValues" color="7" fill="1" visible="yes" active="no"/>
 <layer number="29" name="tStop" color="7" fill="3" visible="no" active="no"/>
 <layer number="30" name="bStop" color="7" fill="6" visible="no" active="no"/>
@@
 <layer number="35" name="tGlue" color="7" fill="4" visible="no" active="no"/>
 <layer number="36" name="bGlue" color="7" fill="5" visible="no" active="no"/>
-<layer number="37" name="tTest" color="7" fill="1" visible="no" active="no"/>
-<layer number="38" name="bTest" color="7" fill="1" visible="no" active="no"/>
+<layer number="37" name="tTest" color="7" fill="1" visible="yes" active="no"/>
+<layer number="38" name="bTest" color="7" fill="1" visible="yes" active="no"/>
 <layer number="39" name="tKeepout" color="4" fill="11" visible="no" active="no"/>
 <layer number="40" name="bKeepout" color="1" fill="11" visible="no" active="no"/>
@@
 <layer number="44" name="Drills" color="7" fill="1" visible="no" active="no"/>
 <layer number="45" name="Holes" color="7" fill="1" visible="no" active="no"/>
-<layer number="46" name="Milling" color="3" fill="1" visible="no" active="no"/>
-<layer number="47" name="Measures" color="7" fill="1" visible="no" active="no"/>
-<layer number="48" name="Document" color="7" fill="1" visible="no" active="no"/>
-<layer number="49" name="Reference" color="7" fill="1" visible="no" active="no"/>
-<layer number="50" name="dxf" color="7" fill="1" visible="no" active="no"/>
-<layer number="51" name="tDocu" color="15" fill="1" visible="no" active="no"/>
-<layer number="52" name="bDocu" color="7" fill="1" visible="no" active="no"/>
-<layer number="53" name="tGND_GNDA" color="7" fill="9" visible="no" active="no"/>
-<layer number="54" name="bGND_GNDA" color="1" fill="9" visible="no" active="no"/>
-<layer number="56" name="wert" color="7" fill="1" visible="no" active="no"/>
-<layer number="57" name="tCAD" color="7" fill="1" visible="no" active="no"/>
-<layer number="59" name="tCarbon" color="7" fill="1" visible="no" active="no"/>
-<layer number="60" name="bCarbon" color="7" fill="1" visible="no" active="no"/>
+<layer number="46" name="Milling" color="3" fill="1" visible="yes" active="no"/>
+<layer number="47" name="Measures" color="7" fill="1" visible="yes" active="no"/>
+<layer number="48" name="Document" color="7" fill="1" visible="yes" active="no"/>
+<layer number="49" name="Reference" color="7" fill="1" visible="yes" active="no"/>
+<layer number="50" name="dxf" color="7" fill="1" visible="yes" active="no"/>
+<layer number="51" name="tDocu" color="15" fill="1" visible="yes" active="no"/>
+<layer number="52" name="bDocu" color="7" fill="1" visible="yes" active="no"/>
+<layer number="53" name="tGND_GNDA" color="7" fill="9" visible="yes" active="no"/>
+<layer number="54" name="bGND_GNDA" color="1" fill="9" visible="yes" active="no"/>
+<layer number="56" name="wert" color="7" fill="1" visible="yes" active="no"/>
+<layer number="57" name="tCAD" color="7" fill="1" visible="yes" active="no"/>
+<layer number="59" name="tCarbon" color="7" fill="1" visible="yes" active="no"/>
+<layer number="60" name="bCarbon" color="7" fill="1" visible="yes" active="no"/>
 <layer number="90" name="Modules" color="5" fill="1" visible="yes" active="yes"/>
 <layer number="91" name="Nets" color="2" fill="1" visible="yes" active="yes"/>
@@
 <part name="VD17" library="diode" deviceset="ZENER-DIODE" device="SOD80C"/>
 <part name="VT18" library="transistor-npn" deviceset="BC849*" device="SMD" value=""/>
-<part name="R35" library="rcl" deviceset="R-EU_" device="R0805"/>
+<part name="R35" library="rcl" deviceset="R-EU_" device="M1206"/>
 <part name="R36" library="rcl" deviceset="R-EU_" device="0207/12"/>
 <part name="GND19" library="supply1" deviceset="GND" device=""/>
 <part name="VD18" library="diode" deviceset="ZENER-DIODE" device="SOD80C"/>
 <part name="VT19" library="transistor-npn" deviceset="BC849*" device="SMD" value=""/>
-<part name="R37" library="rcl" deviceset="R-EU_" device="R0805"/>
+<part name="R37" library="rcl" deviceset="R-EU_" device="0204/7"/>
 <part name="R38" library="rcl" deviceset="R-EU_" device="0207/12"/>
 <part name="GND20" library="supply1" deviceset="GND" device=""/>
 <part name="VD19" library="diode" deviceset="ZENER-DIODE" device="SOD80C"/>
 <part name="VT20" library="transistor-npn" deviceset="BC849*" device="SMD" value=""/>
-<part name="R39" library="rcl" deviceset="R-EU_" device="R0805"/>
+<part name="R39" library="rcl" deviceset="R-EU_" device="R1206W"/>
 <part name="R40" library="rcl" deviceset="R-EU_" device="0207/12"/>
 <part name="GND21" library="supply1" deviceset="GND" device=""/>

Commit message: .
Parts:
- R37: device rcl:R-EU_0204/7 -> rcl:R-EU_R0805
- R39: device rcl:R-EU_R1206W -> rcl:R-EU_R0805
- R41, R43, R45: device rcl:R-EU_R0805 -> rcl:R-EU_R1206W
Changed lines of the file:
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@@
 <part name="VD18" library="diode" deviceset="ZENER-DIODE" device="SOD80C"/>
 <part name="VT19" library="transistor-npn" deviceset="BC849*" device="SMD" value=""/>
-<part name="R37" library="rcl" deviceset="R-EU_" device="0204/7"/>
+<part name="R37" library="rcl" deviceset="R-EU_" device="R0805"/>
 <part name="R38" library="rcl" deviceset="R-EU_" device="0207/12"/>
 <part name="GND20" library="supply1" deviceset="GND" device=""/>
 <part name="VD19" library="diode" deviceset="ZENER-DIODE" device="SOD80C"/>
 <part name="VT20" library="transistor-npn" deviceset="BC849*" device="SMD" value=""/>
-<part name="R39" library="rcl" deviceset="R-EU_" device="R1206W"/>
+<part name="R39" library="rcl" deviceset="R-EU_" device="R0805"/>
 <part name="R40" library="rcl" deviceset="R-EU_" device="0207/12"/>
 <part name="GND21" library="supply1" deviceset="GND" device=""/>
 <part name="VD20" library="diode" deviceset="ZENER-DIODE" device="SOD80C"/>
 <part name="VT21" library="transistor-npn" deviceset="BC849*" device="SMD" value=""/>
-<part name="R41" library="rcl" deviceset="R-EU_" device="R0805"/>
+<part name="R41" library="rcl" deviceset="R-EU_" device="R1206W"/>
 <part name="R42" library="rcl" deviceset="R-EU_" device="0207/12"/>
 <part name="GND22" library="supply1" deviceset="GND" device=""/>
 <part name="VD21" library="diode" deviceset="ZENER-DIODE" device="SOD80C"/>
 <part name="VT22" library="transistor-npn" deviceset="BC849*" device="SMD" value=""/>
-<part name="R43" library="rcl" deviceset="R-EU_" device="R0805"/>
+<part name="R43" library="rcl" deviceset="R-EU_" device="R1206W"/>
 <part name="R44" library="rcl" deviceset="R-EU_" device="0207/12"/>
 <part name="GND23" library="supply1" deviceset="GND" device=""/>
 <part name="VD22" library="diode" deviceset="ZENER-DIODE" device="SOD80C"/>
 <part name="VT23" library="transistor-npn" deviceset="BC849*" device="SMD" value=""/>
-<part name="R45" library="rcl" deviceset="R-EU_" device="R0805"/>
+<part name="R45" library="rcl" deviceset="R-EU_" device="R1206W"/>
 <part name="R46" library="rcl" deviceset="R-EU_" device="0207/12"/>
 <part name="GND24" library="supply1" deviceset="GND" device=""/>
