File: EAGLE/in3watch.sch (EAGLE design)
At the start: 300 parts, among them IC1 74HC595D, IC2 74HC595D, IC3 74HC595D, IC4 74HC595D, IC5 74HC595D, IC6 74HC595D, IC7 74HC595D, J3 J5MM

Commit message: .
Parts:
- added C11, C12, C13: (no value), rcl:C-EUC0805
- R78: device rcl:R-EU_0207/12 -> rcl:R-EU_0207/15
Connections:
- removed net N$84: R78.1, VT39.C
- new net N$77: N26.A, R78.1
- net +100V: now also R78.2; no longer N26.A
- net +5V: now also C11.1, C12.1, C13.1
- net C13: now also VT39.C; no longer R78.2
- net GND: now also C11.2, C12.2, C13.2
Other:
- moved on the sheet: C1, C10, C2, C9, N26

Commit message: .
Parts:
- R81: device rcl:R-EU_R1206W -> rcl:R-EU_R0805
Changed lines of the file:
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@@
 <part name="VD40" library="diode" deviceset="ZENER-DIODE" device="SOD80C"/>
 <part name="VT41" library="transistor-npn" deviceset="BC849*" device="SMD" value=""/>
-<part name="R81" library="rcl" deviceset="R-EU_" device="R1206W"/>
+<part name="R81" library="rcl" deviceset="R-EU_" device="R0805"/>
 <part name="R82" library="rcl" deviceset="R-EU_" device="0207/12"/>
 <part name="GND47" library="supply1" deviceset="GND" device=""/>
@@
 <instance part="N24" gate="G$1" x="96.52" y="119.38"/>
 <instance part="N25" gate="G$1" x="96.52" y="139.7"/>
-<instance part="N26" gate="G$1" x="104.14" y="109.22"/>
+<instance part="N26" gate="G$1" x="104.14" y="109.22" smashed="yes">
+<attribute name="NAME" x="104.14" y="114.935" size="1.778" layer="95"/>
+<attribute name="VALUE" x="109.855" y="114.935" size="1.778" layer="96"/>
+</instance>
 <instance part="N27" gate="G$1" x="147.32" y="129.54" rot="R90"/>
 <instance part="N28" gate="G$1" x="147.32" y="78.74" rot="R90"/>
@@
 <junction x="76.2" y="180.34"/>
 <pinref part="R78" gate="G$1" pin="2"/>
-</segment>
-</net>
+<junction x="147.32" y="139.7"/>
+</segment>
+</net>

Commit message: .
Other:
- moved on the sheet: C12, C13

Commit message: ..
Parts:
- removed R105: 10k, rcl:R-EU_R1206W
- R109: device rcl:R-EU_R1206W -> rcl:R-EU_R0805
Connections:
- removed net N$73: R105.1, R109.2
- net +5V: now also R109.2
- net +5VISP: no longer R105.2
Other:
- moved on the sheet: J1, R109

Commit message: e1e2
Parts:
- added R105, R111: (no value), rcl:R-EU_R0805
- added R112, R114: (no value), rcl:R-EU_M0805
- added RE1, RE2: (no value), pinhead:PINHD-1X1
- added VD53, VD54: (no value), diode:ZENER-DIODESOD80C
- added VT53, VT54: BC849SMD, transistor-npn:BC849SMD
Connections:
- new net N$113: R114.1, VT54.C
- new net N$116: R105.2, VD54.C, VT54.B
- new net N$73: R112.1, VT53.C
- new net N$84: R111.2, VD53.C, VT53.B
- new net RE1: R111.1, RE1.1
- new net RE2: R105.1, RE2.1
- net E1: now also R112.2
- net E2: now also R114.2
- net GND: now also VD53.A, VD54.A, VT53.E, VT54.E
Changed lines of the file:
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@@
 <part name="C12" library="rcl" deviceset="C-EU" device="C0805"/>
 <part name="C13" library="rcl" deviceset="C-EU" device="C0805"/>
+<part name="VT53" library="transistor-npn" deviceset="BC849*" device="SMD" value=""/>
+<part name="R111" library="rcl" deviceset="R-EU_" device="R0805"/>
+<part name="R112" library="rcl" deviceset="R-EU_" device="M0805"/>
+<part name="GND67" library="supply1" deviceset="GND" device=""/>
+<part name="VD53" library="diode" deviceset="ZENER-DIODE" device="SOD80C"/>
+<part name="VT54" library="transistor-npn" deviceset="BC849*" device="SMD" value=""/>
+<part name="R105" library="rcl" deviceset="R-EU_" device="R0805"/>
+<part name="R114" library="rcl" deviceset="R-EU_" device="M0805"/>
+<part name="GND68" library="supply1" deviceset="GND" device=""/>
+<part name="VD54" library="diode" deviceset="ZENER-DIODE" device="SOD80C"/>
+<part name="RE1" library="pinhead" deviceset="PINHD-1X1" device=""/>
+<part name="RE2" library="pinhead" deviceset="PINHD-1X1" device=""/>
 </parts>
 <sheets>
@@
 <attribute name="VALUE" x="127.889" y="92.202" size="1.778" layer="96" rot="R90"/>
 </instance>
+<instance part="VT53" gate="G$1" x="190.5" y="99.06" smashed="yes">
+<attribute name="NAME" x="187.96" y="102.87" size="1.778" layer="95" rot="R180"/>
+<attribute name="VALUE" x="172.72" y="91.44" size="1.778" layer="96"/>
+</instance>
+<instance part="R111" gate="G$1" x="177.8" y="99.06" smashed="yes">
+<attribute name="NAME" x="176.53" y="100.5586" size="1.778" layer="95"/>
+<attribute name="VALUE" x="173.99" y="95.758" size="1.778" layer="96"/>
+</instance>
+<instance part="R112" gate="G$1" x="200.66" y="106.68" smashed="yes">
+<attribute name="NAME" x="198.12" y="108.1786" size="1.778" layer="95"/>
+<attribute name="VALUE" x="196.85" y="103.378" size="1.778" layer="96"/>
+</instance>
+<instance part="GND67" gate="1" x="193.04" y="83.82"/>
+<instance part="VD53" gate="G$1" x="185.42" y="93.98" smashed="yes" rot="R90">
+<attribute name="NAME" x="183.388" y="95.885" size="1.778" layer="95" rot="R180"/>
+<attribute name="VALUE" x="188.849" y="92.202" size="1.778" layer="96" rot="R90"/>
+</instance>
+<instance part="VT54" gate="G$1" x="220.98" y="99.06" smashed="yes">
+<attribute name="NAME" x="218.44" y="102.87" size="1.778" layer="95" rot="R180"/>
+<attribute name="VALUE" x="203.2" y="91.44" size="1.778" layer="96"/>
+</instance>
+<instance part="R105" gate="G$1" x="208.28" y="99.06" smashed="yes">
+<attribute name="NAME" x="207.01" y="100.5586" size="1.778" layer="95"/>
+<attribute name="VALUE" x="204.47" y="95.758" size="1.778" layer="96"/>
+</instance>
+<instance part="R114" gate="G$1" x="231.14" y="106.68" smashed="yes">
+<attribute name="NAME" x="228.6" y="108.1786" size="1.778" layer="95"/>
+<attribute name="VALUE" x="227.33" y="103.378" size="1.778" layer="96"/>
+</instance>
+<instance part="GND68" gate="1" x="223.52" y="83.82"/>
+<instance part="VD54" gate="G$1" x="215.9" y="93.98" smashed="yes" rot="R90">
+<attribute name="NAME" x="213.868" y="95.885" size="1.778" layer="95" rot="R180"/>
+<attribute name="VALUE" x="219.329" y="92.202" size="1.778" layer="96" rot="R90"/>
+</instance>
+<instance part="RE1" gate="G$1" x="170.18" y="76.2"/>
+<instance part="RE2" gate="G$1" x="170.18" y="68.58"/>
 </instances>
 <busses>
@@
 <junction x="132.08" y="88.9"/>
 </segment>
+<segment>
+<pinref part="VT53" gate="G$1" pin="E"/>
+<pinref part="GND67" gate="1" pin="GND"/>
+<wire x1="193.04" y1="93.98" x2="193.04" y2="88.9" width="0.1524" layer="91"/>
+<pinref part="VD53" gate="G$1" pin="A"/>
+<wire x1="193.04" y1="88.9" x2="193.04" y2="86.36" width="0.1524" layer="91"/>
+<wire x1="185.42" y1="91.44" x2="185.42" y2="88.9" width="0.1524" layer="91"/>
+<wire x1="185.42" y1="88.9" x2="193.04" y2="88.9" width="0.1524" layer="91"/>
+<junction x="193.04" y="88.9"/>
+</segment>
+<segment>
+<pinref part="VT54" gate="G$1" pin="E"/>
+<pinref part="GND68" gate="1" pin="GND"/>
+<wire x1="223.52" y1="93.98" x2="223.52" y2="88.9" width="0.1524" layer="91"/>
+<pinref part="VD54" gate="G$1" pin="A"/>
+<wire x1="223.52" y1="88.9" x2="223.52" y2="86.36" width="0.1524" layer="91"/>
+<wire x1="215.9" y1="91.44" x2="215.9" y2="88.9" width="0.1524" layer="91"/>
+<wire x1="215.9" y1="88.9" x2="223.52" y2="88.9" width="0.1524" layer="91"/>
+<junction x="223.52" y="88.9"/>
+</segment>
 </net>
 <net name="N$69" class="0">
@@
 </segment>
 </net>
+<net name="N$73" class="0">
+<segment>
+<pinref part="VT53" gate="G$1" pin="C"/>
+<wire x1="193.04" y1="104.14" x2="193.04" y2="106.68" width="0.1524" layer="91"/>
+<pinref part="R112" gate="G$1" pin="1"/>
+<wire x1="193.04" y1="106.68" x2="195.58" y2="106.68" width="0.1524" layer="91"/>
+</segment>
+</net>
+<net name="N$84" class="0">
+<segment>
+<pinref part="VT53" gate="G$1" pin="B"/>
+<pinref part="R111" gate="G$1" pin="2"/>
+<wire x1="187.96" y1="99.06" x2="185.42" y2="99.06" width="0.1524" layer="91"/>
+<pinref part="VD53" gate="G$1" pin="C"/>
+<wire x1="185.42" y1="99.06" x2="182.88" y2="99.06" width="0.1524" layer="91"/>
+<wire x1="185.42" y1="96.52" x2="185.42" y2="99.06" width="0.1524" layer="91"/>
+<junction x="185.42" y="99.06"/>
+</segment>
+</net>
+<net name="E1" class="0">
+<segment>
+<pinref part="R112" gate="G$1" pin="2"/>
+<wire x1="205.74" y1="106.68" x2="210.82" y2="106.68" width="0.1524" layer="91"/>
+<label x="205.74" y="106.68" size="1.778" layer="95"/>
+</segment>
+</net>
+<net name="RE1" class="0">
+<segment>
+<pinref part="R111" gate="G$1" pin="1"/>
+<wire x1="172.72" y1="99.06" x2="167.64" y2="99.06" width="0.1524" layer="91"/>
+<label x="172.72" y="99.06" size="1.778" layer="95" rot="MR0"/>
+</segment>
+<segment>
+<pinref part="RE1" gate="G$1" pin="1"/>
+<wire x1="167.64" y1="76.2" x2="154.94" y2="76.2" width="0.1524" layer="91"/>
+<label x="154.94" y="76.2" size="1.778" layer="95"/>
+</segment>
+</net>
+<net name="N$113" class="0">
+<segment>
+<pinref part="VT54" gate="G$1" pin="C"/>
+<wire x1="223.52" y1="104.14" x2="223.52" y2="106.68" width="0.1524" layer="91"/>
+<pinref part="R114" gate="G$1" pin="1"/>
+<wire x1="223.52" y1="106.68" x2="226.06" y2="106.68" width="0.1524" layer="91"/>
+</segment>
+</net>
+<net name="N$116" class="0">
+<segment>
+<pinref part="VT54" gate="G$1" pin="B"/>
+<pinref part="R105" gate="G$1" pin="2"/>
+<wire x1="218.44" y1="99.06" x2="215.9" y2="99.06" width="0.1524" layer="91"/>
+<pinref part="VD54" gate="G$1" pin="C"/>
+<wire x1="215.9" y1="99.06" x2="213.36" y2="99.06" width="0.1524" layer="91"/>
+<wire x1="215.9" y1="96.52" x2="215.9" y2="99.06" width="0.1524" layer="91"/>
+<junction x="215.9" y="99.06"/>
+</segment>
+</net>
+<net name="RE2" class="0">
+<segment>
+<pinref part="R105" gate="G$1" pin="1"/>
+<wire x1="203.2" y1="99.06" x2="198.12" y2="99.06" width="0.1524" layer="91"/>
+<label x="203.2" y="99.06" size="1.778" layer="95" rot="MR0"/>
+</segment>
+<segment>
+<pinref part="RE2" gate="G$1" pin="1"/>
+<wire x1="167.64" y1="68.58" x2="154.94" y2="68.58" width="0.1524" layer="91"/>
+<label x="154.94" y="68.58" size="1.778" layer="95"/>
+</segment>
+</net>
+<net name="E2" class="0">
+<segment>
+<pinref part="R114" gate="G$1" pin="2"/>
+<wire x1="236.22" y1="106.68" x2="241.3" y2="106.68" width="0.1524" layer="91"/>
+<label x="236.22" y="106.68" size="1.778" layer="95"/>
+</segment>
+</net>

Commit message: .
Parts:
- N27: value IN-3 -> IN-33; device in3:IN-3 -> in3-mod:IN-33
Changed lines of the file:
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@@
 <part name="N25" library="in3-mod" deviceset="IN-3" device="1"/>
 <part name="N26" library="in3" deviceset="IN-3" device=""/>
-<part name="N27" library="in3" deviceset="IN-3" device=""/>
+<part name="N27" library="in3-mod" deviceset="IN-3" device="3"/>
 <part name="N28" library="in3" deviceset="IN-3" device=""/>
 <part name="N29" library="in3" deviceset="IN-3" device=""/>

Commit message: +dot2
Parts:
- R48: device rcl:R-EU_0207/12 -> rcl:R-EU_0207/10
Changed lines of the file:
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@@
 <part name="VT24" library="transistor-npn" deviceset="BC849*" device="SMD" value=""/>
 <part name="R47" library="rcl" deviceset="R-EU_" device="R0805"/>
-<part name="R48" library="rcl" deviceset="R-EU_" device="0207/12"/>
+<part name="R48" library="rcl" deviceset="R-EU_" device="0207/10"/>
 <part name="GND25" library="supply1" deviceset="GND" device=""/>
 <part name="VD24" library="diode" deviceset="ZENER-DIODE" device="SOD80C"/>
