File: EAGLE/in3watch.brd (EAGLE design)
At the start: 297 parts, among them IC1 74HC595D, IC2 74HC595D, IC3 74HC595D, IC4 74HC595D, IC5 74HC595D, IC6 74HC595D, IC7 74HC595D, J3 J5MM

Commit message: ..>
Parts:
- moved R65 4.72 mm to (-15.9, -14.0), turned to 270 degrees
- moved R101 3.00 mm to (-108.1, 16.4), turned to 0 degrees
- moved R57 1.90 mm to (-23.8, 32.1), turned to 180 degrees
- moved R89 1.59 mm to (-80.6, 4.35)
- moved R83 1.31 mm to (-78.6, 22.2)
Routing:
- net GND: track 1117.8 -> 1320.1 mm, vias 6 -> 8
- net RC9: track 0.00 -> 40.7 mm
- net RC10: track 0.00 -> 33.0 mm
- net RC8: track 0.00 -> 25.0 mm
- net RD4: track 2.62 -> 20.9 mm
- net RC7: track 0.00 -> 15.1 mm
- net N$109: track 12.8 -> 15.2 mm
- net RD12: track 5.78 -> 3.95 mm
- net RD6: track 7.32 -> 8.90 mm
- net N$97: track 21.3 -> 19.7 mm
- net N$61: track 6.26 -> 5.09 mm
- net N$69: track 4.63 -> 5.36 mm

Commit message: .
Parts:
- moved VD32 5.85 mm to (-13.3, -3.81), turned to 180 degrees
- moved VD31 5.41 mm to (-13.3, 10.2), turned to 180 degrees
- moved VD38 5.39 mm to (-48.6, 17.8), turned to 90 degrees
- moved VD30 4.85 mm to (-10.2, 13.0), turned to 0 degrees
- moved R59 4.32 mm to (-11.1, 21.6), turned to 180 degrees
- moved R63 4.07 mm to (-14.9, -0.95)
- moved R61 4.04 mm to (-14.6, 13.0)
- moved VT32 1.71 mm to (-14.0, -6.99), turned to 180 degrees
- moved R75 1.62 mm to (-43.5, 14.0)
- moved VT31 1.42 mm to (-14.0, 6.99), turned to 180 degrees
- moved VT30 1.14 mm to (-11.1, 17.1), turned to 0 degrees
- moved VD39 0.32 mm to (-35.9, -4.76)
- moved R78 0.32 mm to (-35.9, 9.53)
- moved R73 0.32 mm to (-46.0, 0.64)
Connections:
- net N$17 renamed +100V
Routing:
- net GND: track 1320.1 -> 1393.6 mm
- net +100V: track 866.9 -> 935.3 mm, vias 4 -> 6
- net RC11: track 0.00 -> 41.5 mm
- net RC10: track 33.0 -> 50.1 mm
- net RC9: track 40.7 -> 57.3 mm
- net RC7: track 15.1 -> 31.1 mm
- net RC13: track 0.00 -> 14.4 mm
- net RC8: track 25.0 -> 39.4 mm
- net N$63: track 4.49 -> 10.7 mm
- net RC4: track 19.1 -> 14.1 mm
- net C13: track 0.00 -> 3.29 mm
- net RC6: track 27.1 -> 24.2 mm
- net RC5: track 14.9 -> 12.9 mm
- net N$67: track 4.78 -> 3.99 mm
- net N$66: track 2.55 -> 2.03 mm
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
Commit message: ..
Parts:
- R75: device rcl:R0805 -> rcl:R1206W
- moved VD38 6.99 mm to (-44.1, 12.4), turned to 0 degrees
- moved R75 6.61 mm to (-39.7, 8.57), turned to 90 degrees
- moved R77 4.69 mm to (-32.4, -0.64), turned to 270 degrees
- moved R55 3.72 mm to (-27.3, 29.5)
- moved VT38 1.42 mm to (-44.1, 16.2), turned to 0 degrees
- moved IC4 1.42 mm to (-28.9, 22.4)
- moved VT28 0.71 mm to (-30.5, 33.0)
- moved VD28 0.63 mm to (-34.3, 33.3)
- moved IC5 0.41 mm to (-28.9, 7.51), turned to 0 degrees
- moved VD39 0.32 mm to (-35.9, -4.45)
Routing:
- net RC12: track 0.00 -> 32.3 mm
- net RC10: track 50.1 -> 38.7 mm
- net RC9: track 57.3 -> 46.7 mm
- net RC13: track 14.4 -> 4.76 mm
- net RC11: track 41.5 -> 32.7 mm
- net N$83: track 0.00 -> 7.31 mm
- net RC8: track 39.4 -> 32.1 mm
- net RC2: track 13.3 -> 9.59 mm
- net RC7: track 31.1 -> 29.0 mm
- net N$82: track 0.00 -> 1.92 mm
- net RDATA_MOSI_D11: track 109.5 -> 108.1 mm
- net N$59: track 5.61 -> 6.93 mm
- net GND: track 1393.6 -> 1394.8 mm
- net RC6: track 24.2 -> 25.0 mm
- net RC5: track 12.9 -> 13.7 mm
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
Commit message: ...
Parts:
- added J6: (no value), rcl:R1206W
- moved IC5 0.95 mm to (-28.0, 7.51)
Connections:
- new net N$17: IC5.14, J6.2
- net SER5: now also J6.1; no longer IC5.14
Routing:
- net RLATCH_D10: track 269.3 -> 301.9 mm
- net RCLOCK_MISO_D12: track 205.2 -> 232.9 mm
- net +5V: track 443.2 -> 465.4 mm
- net SER5: track 0.00 -> 8.54 mm
- net N$17: track 0.00 -> 7.84 mm
- net GND: track 1394.8 -> 1397.9 mm
- net SER4: track 81.5 -> 80.2 mm
- net RC7: track 29.0 -> 28.3 mm

Commit message: .
Parts:
- R56: device rcl:0207/12 -> rcl:0207/10
- moved R57 4.51 mm to (-20.3, 29.2), turned to 90 degrees
- moved VD37 4.02 mm to (-48.9, 0.95), turned to 0 degrees
- moved R73 1.71 mm to (-44.5, 1.27)
- moved R75 1.14 mm to (-40.6, 9.21)
- moved VT28 1.00 mm to (-31.4, 33.3)
- moved R77 1.00 mm to (-32.1, -1.59)
- moved R74 0.90 mm to (-47.6, 9.53)
- moved VD28 0.63 mm to (-34.9, 33.3)
- moved R78 0.32 mm to (-35.9, 9.21)
Routing:
- net RD1: track 3.82 -> 88.1 mm, vias 1 -> 2
- net GND: track 1397.9 -> 1447.4 mm
- net SER4: track 80.2 -> 84.5 mm
- net RC3: track 12.1 -> 9.48 mm
- net +100V: track 935.2 -> 933.1 mm
- net N$81: track 5.92 -> 4.49 mm
- net RC11: track 32.7 -> 31.5 mm
- net N$61: track 5.09 -> 3.98 mm
- net N$83: track 7.31 -> 6.27 mm
- net RC13: track 5.15 -> 5.97 mm
- net RC12: track 32.4 -> 33.1 mm
- net N$59: track 6.93 -> 7.65 mm
- net C11: track 5.39 -> 4.80 mm
- net N$80: track 2.44 -> 1.90 mm
- net N$85: track 6.29 -> 5.76 mm
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
Commit message: ..
Parts:
- R76: device rcl:0207/12 -> rcl:0207/10
- moved R53 4.97 mm to (-43.2, 28.9)
- moved IC4 4.14 mm to (-33.0, 22.8)
- moved R75 4.14 mm to (-44.8, 9.53)
- moved VT27 2.69 mm to (-46.0, 33.0)
- moved VD38 2.29 mm to (-46.0, 13.7)
- moved VD27 2.13 mm to (-49.5, 34.0)
- moved VT38 2.01 mm to (-46.0, 16.8)
- moved VD28 1.59 mm to (-34.0, 34.6)
- moved R76 0.90 mm to (-47.9, 23.8)
- moved VT37 0.90 mm to (-46.7, 5.08)
- moved VT28 0.71 mm to (-30.8, 33.7)
- moved R73 0.71 mm to (-44.1, 0.64)
- moved VD37 0.32 mm to (-48.9, 0.64)
Routing:
- net RCLOCK_MISO_D12: track 232.9 -> 297.9 mm, vias 4 -> 5
- net +5V: track 465.4 -> 506.6 mm, vias 10 -> 11
- net RLATCH_D10: track 301.9 -> 338.6 mm, vias 3 -> 4
- net GND: track 1447.4 -> 1476.1 mm
- net RC1: track 0.00 -> 18.9 mm
- net SER4: track 84.5 -> 99.0 mm
- net RD1: track 88.1 -> 94.4 mm
- net RC5: track 14.1 -> 18.4 mm
- net RC6: track 25.6 -> 29.8 mm
- net SER5: track 8.54 -> 12.7 mm
- net RC4: track 14.0 -> 18.1 mm
- net RB12: track 18.6 -> 14.5 mm
- net RC3: track 9.48 -> 13.5 mm
- net RC2: track 9.59 -> 13.3 mm
- net RC12: track 33.1 -> 36.4 mm
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
Commit message: ...
Parts:
- moved IC6 1.90 mm to (-84.5, 14.0)
- moved R77 1.80 mm to (-33.3, -2.86)
- moved VD39 1.27 mm to (-37.1, -4.45)
- moved R89 1.27 mm to (-80.6, 3.08)
- moved R87 1.00 mm to (-77.0, 7.84)
- moved VT39 0.95 mm to (-37.1, -0.64)
Routing:
- net RLATCH_D10: track 338.6 -> 281.8 mm, vias 4 -> 5
- net +5V: track 506.6 -> 449.9 mm, vias 11 -> 12
- net RD3: track 7.24 -> 13.3 mm
- net GND: track 1476.1 -> 1478.3 mm
- net SER6: track 5.50 -> 7.41 mm
- net RD8: track 36.6 -> 34.7 mm
- net RD7: track 39.4 -> 37.5 mm
- net RD2: track 10.1 -> 12.0 mm
- net RD9: track 39.0 -> 37.1 mm
- net RCLOCK_MISO_D12: track 297.9 -> 299.7 mm
- net RC13: track 5.97 -> 7.77 mm
- net RD4: track 20.9 -> 22.2 mm
- net N$97: track 19.7 -> 18.5 mm
- net RC12: track 36.4 -> 37.7 mm
- net RC11: track 30.8 -> 31.7 mm
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
Commit message: .....
Parts:
- added C10, C9: (no value), rcl:C0805
- moved VD51 5.20 mm to (-105.6, 11.9), turned to 270 degrees
- moved R101 1.62 mm to (-106.5, 16.8)
- moved VT51 0.74 mm to (-105.3, 6.76), turned to 180 degrees
- moved R53 0.71 mm to (-43.8, 29.2)
Connections:
- net +5V: now also C10.1, C9.1
- net GND: now also C10.2, C9.2
Routing:
- net +5V: track 449.9 -> 417.9 mm
- net GND: track 1478.3 -> 1491.7 mm, vias 8 -> 6
- net N$109: track 15.2 -> 12.6 mm
- net N$108: track 1.81 -> 3.90 mm
- net RD12: track 3.95 -> 2.23 mm
- net N$57: track 6.78 -> 6.12 mm
