File: EAGLE/in3watch.brd (EAGLE design)
At the start: 300 parts, among them IC1 74HC595D, IC2 74HC595D, IC3 74HC595D, IC4 74HC595D, IC5 74HC595D, IC6 74HC595D, IC7 74HC595D, J3 J5MM

Commit message: .
Parts:
- added C11, C12, C13: (no value), rcl:C0805
- R78: device rcl:0207/12 -> rcl:0207/15
- moved R78 15.0 mm to (-21.0, 10.8), turned to 315 degrees
- moved VD30 6.16 mm to (-6.67, 18.1), turned to 270 degrees
- moved VD31 5.54 mm to (-8.26, 12.4)
- moved VT31 5.02 mm to (-9.21, 8.57)
- moved R55 4.07 mm to (-24.1, 32.1)
- moved R49 3.93 mm to (8.57, 13.3)
- moved IC4 3.55 mm to (-31.4, 25.9), turned to 275 degrees
- moved R89 2.86 mm to (-80.6, 0.22)
- moved R87 2.56 mm to (-74.5, 7.53)
- moved R61 2.13 mm to (-12.7, 14.0), turned to 180 degrees
- moved VD28 1.85 mm to (-35.6, 35.6)
- moved VT28 1.80 mm to (-32.1, 34.9)
- moved R57 1.62 mm to (-18.7, 28.9)
- moved R56 1.42 mm to (-32.7, 37.1)
- moved VT25 1.42 mm to (11.4, 17.8)
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Connections:
- removed net N$84: R78.1, VT39.C
- new net N$77: N26.A, R78.1
- net +100V: now also R78.2; no longer N26.A
- net +5V: now also C11.1, C12.1, C13.1
- net C13: now also VT39.C; no longer R78.2
- net GND: now also C11.2, C12.2, C13.2
Routing:
- net SER6: track 7.41 -> 80.4 mm, vias 1 -> 2
- net RB12: track 14.5 -> 61.8 mm, vias 0 -> 2
- net GND: track 1491.7 -> 1528.5 mm
- net +5V: track 417.9 -> 444.6 mm
- net N$64: track 2.03 -> 19.8 mm
- net +100V: track 933.1 -> 916.1 mm
- net C13: track 3.32 -> 17.3 mm, vias 0 -> 1
- net RB13: track 4.47 -> 17.1 mm, vias 0 -> 2
- net SER4: track 99.4 -> 88.0 mm
- net N$63: track 10.7 -> 5.89 mm
- net N$59: track 6.92 -> 11.4 mm
- net RCLOCK_MISO_D12: track 299.7 -> 303.3 mm
- net N$95: track 10.3 -> 6.84 mm
- net RLATCH_D10: track 281.8 -> 285.2 mm
- net N$91: track 19.1 -> 22.3 mm
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
Commit message: ..
Parts:
- moved C12 0.64 mm to (32.4, 13.7)
Routing:
- net SER4: track 88.0 -> 89.1 mm
- net C12: track 6.66 -> 5.83 mm
- net RLATCH_D10: track 285.2 -> 285.9 mm

Commit message: ...
Parts:
- moved VD1 13.1 mm to (69.7, 37.2), turned to 135 degrees
- moved C12 8.89 mm to (23.5, 13.7), turned to 270 degrees
- moved VD12 7.36 mm to (72.1, 14.7), turned to 0 degrees
- moved VT1 6.51 mm to (72.4, 34.7), turned to 135 degrees
- moved C2 6.22 mm to (94.0, 14.5), turned to 90 degrees
- moved R41 3.62 mm to (20.3, 3.49)
- moved R23 2.88 mm to (76.3, 12.4)
- moved VD14 2.58 mm to (21.6, 33.2), turned to 180 degrees
- moved VT12 2.50 mm to (71.4, 18.5), turned to 0 degrees
- moved R39 2.25 mm to (22.9, 4.60)
- moved R52 2.13 mm to (2.22, 27.3)
- moved R1 1.78 mm to (82.2, 32.6), turned to 0 degrees
- moved VT10 1.62 mm to (73.1, -5.40)
- moved VD10 1.59 mm to (69.3, -5.08)
- moved R57 1.27 mm to (-20.0, 28.9)
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Routing:
- net +5V: track 444.4 -> 500.7 mm, vias 12 -> 13
- net GND: track 1528.5 -> 1509.4 mm, vias 6 -> 8
- net N$2: track 4.44 -> 16.7 mm
- net N$45: track 48.9 -> 44.4 mm
- net RB8: track 2.67 -> 6.95 mm
- net N$13: track 10.1 -> 5.84 mm
- net RDATA_MOSI_D11: track 108.1 -> 111.7 mm
- net RA12: track 8.03 -> 5.16 mm
- net +100V: track 916.1 -> 918.9 mm
- net N$43: track 64.7 -> 67.1 mm
- net RB7: track 5.32 -> 2.99 mm
- net RCLOCK_MISO_D12: track 303.1 -> 304.9 mm
- net N$9: track 18.2 -> 20.0 mm
- net N$30: track 17.6 -> 15.9 mm
- net RC2: track 12.6 -> 10.9 mm
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
Commit message: .
Parts:
- R81: device rcl:R1206W -> rcl:R0805
- moved VD18 11.2 mm to (45.2, 12.4), turned to 180 degrees
- moved VD42 10.5 mm to (-80.4, 35.7), turned to 90 degrees
- moved VT18 5.02 mm to (44.8, 9.21), turned to 180 degrees
- moved VT42 3.38 mm to (-76.7, 34.9), turned to 90 degrees
- moved R35 1.93 mm to (40.1, 0.32)
- moved R1 0.95 mm to (81.3, 32.6)
- moved VD25 0.95 mm to (7.94, 18.1)
- moved R81 0.71 mm to (-82.1, 30.1)
- moved R19 0.10 mm to (76.7, -1.91)
Routing:
- net N$39: track 24.8 -> 12.6 mm
- net GND: track 1509.4 -> 1499.6 mm
- net N$91: track 22.3 -> 13.6 mm
- net +100V: track 918.9 -> 916.6 mm
- net RB5: track 16.5 -> 18.4 mm
- net +5V: track 500.7 -> 502.3 mm
- net RA1: track 11.9 -> 13.2 mm
- net RA9: track 45.1 -> 43.9 mm
- net N$90: track 2.66 -> 3.68 mm
- net N$2: track 16.7 -> 15.7 mm
- net N$41: track 13.5 -> 14.2 mm
- net RD2: track 12.0 -> 12.5 mm
- net N$89: track 6.88 -> 6.37 mm

Commit message: .
Parts:
- moved R85 10.4 mm to (-74.2, 14.9)
- moved VD43 6.47 mm to (-72.5, 27.1), turned to 180 degrees
- moved VT43 1.79 mm to (-72.9, 23.4), turned to 180 degrees
- moved VT14 0.66 mm to (16.9, 36.8), turned to 180 degrees
Routing:
- net GND: track 1499.6 -> 1466.7 mm
- net RD4: track 22.7 -> 12.3 mm
- net N$93: track 5.49 -> 14.1 mm
- net +100V: track 916.6 -> 913.9 mm
- net N$16: track 4.37 -> 2.48 mm
- net N$30: track 15.9 -> 17.4 mm
- net N$92: track 1.98 -> 2.66 mm

Commit message: .
Parts:
- moved C12 1.27 mm to (24.8, 13.7)
- moved VD15 0.95 mm to (33.1, 31.3)
Routing:
- net GND: track 1466.7 -> 1532.6 mm, vias 8 -> 9
- net RLATCH_D10: track 286.1 -> 316.3 mm
- net +5V: track 502.3 -> 525.0 mm, vias 13 -> 14
- net SER6: track 80.8 -> 66.1 mm
- net RD10: track 51.3 -> 48.7 mm
- net RCLOCK_MISO_D12: track 305.3 -> 307.8 mm
- net SER4: track 89.9 -> 92.2 mm
- net B13: track 25.5 -> 27.7 mm
- net RD9: track 37.1 -> 35.0 mm
- net +100V: track 913.9 -> 915.8 mm

Commit message: .
Parts:
- moved VD34 6.55 mm to (-17.5, -27.9), turned to 270 degrees
- moved R73 4.27 mm to (-47.0, -2.54), turned to 90 degrees
- moved VT39 3.27 mm to (-38.7, -3.49)
- moved VD39 3.00 mm to (-38.7, -6.99)
- moved R67 2.56 mm to (-17.6, -23.3)
- moved VT34 1.14 mm to (-20.6, -27.9), turned to 270 degrees
- moved R77 0.32 mm to (-33.3, -2.54), turned to 0 degrees
Routing:
- net GND: track 1532.6 -> 1543.3 mm, vias 9 -> 10
- net RC12: track 37.7 -> 47.0 mm
- net RLATCH_D10: track 316.3 -> 322.9 mm
- net RC11: track 31.7 -> 37.4 mm
- net N$71: track 7.02 -> 4.17 mm
- net N$85: track 5.02 -> 7.73 mm
- net C13: track 17.3 -> 19.9 mm
- net RC8: track 31.7 -> 29.1 mm
- net RB12: track 61.8 -> 59.8 mm
- net RD1: track 94.4 -> 93.1 mm
- net RC9: track 47.1 -> 46.4 mm

Commit message: .
Parts:
- moved C1 9.56 mm to (88.6, 26.4), turned to 135 degrees
- moved R84 2.25 mm to (-70.6, 37.5)
Routing:
- net GND: track 1543.3 -> 1789.0 mm, vias 10 -> 13
- net RESET: track 24.2 -> 28.7 mm
- net RD2: track 12.5 -> 16.8 mm
- net SER6: track 66.1 -> 68.8 mm
- net D3: track 5.65 -> 3.41 mm
- net N$90: track 3.96 -> 2.10 mm
- net +5V: track 525.0 -> 526.3 mm
- net N$91: track 13.6 -> 14.6 mm
- net +100V: track 915.8 -> 915.1 mm
