File: EAGLE/in3watch.brd (EAGLE design)
At the start: 303 parts, among them IC1 74HC595D, IC2 74HC595D, IC3 74HC595D, IC4 74HC595D, IC5 74HC595D, IC6 74HC595D, IC7 74HC595D, J3 J5MM

Commit message: ..
Parts:
- moved VT6 1.62 mm to (101.3, -11.3)
- moved VD6 1.27 mm to (98.0, -10.1)
- moved VD45 0.64 mm to (-67.4, -7.94)
- moved VT45 0.64 mm to (-70.6, -7.94)
- moved VD25 0.63 mm to (7.30, 18.1)
- moved VT25 0.63 mm to (10.8, 17.8)
- moved VT16 0.45 mm to (46.3, 35.4)
- moved VT41 0.32 mm to (-87.6, 32.5)
- moved C8 0.32 mm to (57.6, -25.9)
- moved VT20 0.32 mm to (32.7, -31.1)
- moved VD19 0.32 mm to (44.5, -1.27)
- moved VT19 0.32 mm to (44.5, -4.45)
- moved R105 0.32 mm to (23.8, -10.8)
- moved VD20 0.32 mm to (29.1, -30.3)
- moved VD23 0.32 mm to (16.0, -4.29)
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Routing:
- net SER2: track 19.3 -> 26.6 mm
- net +5V: track 526.3 -> 529.5 mm, vias 14 -> 13
- net N$25: track 10.0 -> 11.0 mm
- net SDA: track 71.8 -> 72.6 mm
- net N$52: track 1.80 -> 2.44 mm
- net N$96: track 1.80 -> 2.44 mm
- net SCL: track 61.5 -> 62.1 mm
- net N$24: track 1.67 -> 2.18 mm
Other:
- board outline added: 242.6 x 106.7 mm

Commit message: ..
Parts:
- removed R105: 10k, rcl:R1206W
- R109: device rcl:R1206W -> rcl:R0805
- moved R109 14.2 mm to (33.7, -23.8), turned to 270 degrees
- moved R59 5.79 mm to (-16.8, 20.6)
- moved C4 3.14 mm to (33.3, -11.7)
- moved R51 2.29 mm to (-15.2, 25.1)
- moved VD26 2.03 mm to (-11.7, 27.0)
- moved VT26 1.59 mm to (-7.94, 27.3)
Connections:
- removed net N$73: R105.1, R109.2
- net +5V: now also R109.2
- net +5VISP: no longer R105.2
Routing:
- net RCLOCK_MISO_D12: track 308.2 -> 334.1 mm
- net RC4: track 17.1 -> 11.5 mm
- net N$63: track 5.95 -> 10.3 mm
- net N$73: track 3.69 -> 0.00 mm
- net N$76: track 7.89 -> 4.75 mm
- net +5V: track 529.5 -> 532.6 mm
- net RESET: track 28.7 -> 26.1 mm
- net GND: track 1788.7 -> 1791.1 mm
- net +5VISP: track 4.78 -> 2.62 mm
- net RB13: track 17.0 -> 14.9 mm
- net N$54: track 2.17 -> 2.71 mm
Other:
- board size 242.6 x 106.7 mm -> 233.7 x 96.2 mm

Commit message: .
Parts:
- moved VD48 12.2 mm to (-105.6, -31.2), turned to 90 degrees
- moved R94 11.0 mm to (-89.2, -23.2)
- moved R92 10.0 mm to (-79.9, -27.9)
- moved VD45 9.74 mm to (-74.3, -1.05), turned to 180 degrees
- moved VT48 7.55 mm to (-102.1, -31.8), turned to 90 degrees
- moved VT47 6.44 mm to (-84.7, -21.9), turned to 0 degrees
- moved VT46 6.37 mm to (-76.3, -26.8), turned to 0 degrees
- moved VT45 5.03 mm to (-74.3, -4.54), turned to 180 degrees
- moved R93 4.18 mm to (-81.2, -21.0)
- moved VD46 3.26 mm to (-77.1, -30.3), turned to 0 degrees
- moved R91 3.14 mm to (-68.5, -16.5)
- moved R89 1.59 mm to (-80.6, 1.81)
- moved VD47 1.54 mm to (-85.0, -25.4), turned to 0 degrees
Routing:
- net N$99: track 29.9 -> 12.4 mm
- net N$103: track 6.95 -> 23.9 mm
- net GND: track 1791.1 -> 1805.8 mm
- net D8: track 7.99 -> 21.3 mm
- net N$97: track 17.0 -> 11.1 mm
- net +100V: track 915.1 -> 911.6 mm
- net N$101: track 4.73 -> 7.60 mm
- net RD7: track 37.5 -> 39.7 mm
- net D7: track 7.96 -> 9.84 mm
- net RD6: track 11.1 -> 9.54 mm
- net RD8: track 34.7 -> 33.6 mm
- net N$102: track 2.87 -> 3.48 mm

Commit message: ..
Routing:
- net SCK: track 46.1 -> 42.7 mm

Commit message: 1
Parts:
- moved VD31 6.03 mm to (-14.3, 12.4)
- moved VT31 5.17 mm to (-14.3, 9.53)
- moved R61 3.62 mm to (-16.2, 14.9), turned to 270 degrees
Routing:
- net N$64: track 19.8 -> 14.2 mm
- net GND: track 1805.8 -> 1810.5 mm
- net RC5: track 18.2 -> 15.0 mm
- net N$65: track 5.19 -> 3.51 mm
Changed lines of the file:
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@@
 <element name="R60" library="rcl" package="0207/12" value="" x="-9.8425" y="13.6525" rot="R315"/>
 <element name="VD30" library="diode" package="SOD80C" value="" x="-6.6675" y="18.0975" rot="MR270"/>
-<element name="VT31" library="transistor-npn" package="SOT23-BEC" value="" x="-9.2075" y="8.5725" rot="MR180"/>
-<element name="R61" library="rcl" package="R0805" value="" x="-12.7" y="13.97" rot="MR180"/>
+<element name="VT31" library="transistor-npn" package="SOT23-BEC" value="" x="-14.2875" y="9.525" rot="MR180"/>
+<element name="R61" library="rcl" package="R0805" value="" x="-16.1925" y="14.9225" rot="MR270"/>
 <element name="R62" library="rcl" package="0207/12" value="" x="-8.89" y="-0.9525" rot="R315"/>
-<element name="VD31" library="diode" package="SOD80C" value="" x="-8.255" y="12.3825" rot="MR180"/>
+<element name="VD31" library="diode" package="SOD80C" value="" x="-14.2875" y="12.3825" rot="MR180"/>
 <element name="VT32" library="transistor-npn" package="SOT23-BEC" value="" x="-13.97" y="-6.985" rot="MR180"/>
 <element name="R63" library="rcl" package="R0805" value="" x="-14.9225" y="-0.9525" rot="MR270"/>
@@
 <wire x1="-104.30125" y1="7.8625" x2="-104.30125" y2="9.68625" width="0.6096" layer="16"/>
 <wire x1="-104.30125" y1="9.68625" x2="-104.4575" y2="9.8425" width="0.6096" layer="16"/>
-<wire x1="-8.2575" y1="9.6725" x2="-8.2575" y2="10.68" width="0.6096" layer="16"/>
-<wire x1="-8.2575" y1="10.68" x2="-6.555" y2="12.3825" width="0.6096" layer="16"/>
 <wire x1="-6.6675" y1="16.3975" x2="-6.652621875" y2="15.866521875" width="0.6096" layer="16"/>
-<wire x1="-6.652621875" y1="15.866521875" x2="-6.555" y2="12.3825" width="0.6096" layer="16"/>
 <wire x1="-10.0125" y1="17.1475" x2="-6.6675" y2="16.3975" width="0.6096" layer="16"/>
 <wire x1="7.3025" y1="19.7975" x2="6.145" y2="19.7975" width="0.6096" layer="16"/>
 <wire x1="6.145" y1="19.7975" x2="2.8575" y2="15.875" width="0.6096" layer="16"/>
-<wire x1="2.8575" y1="15.875" x2="-1.27" y2="15.875" width="0.6096" layer="16"/>
-<wire x1="-1.27" y1="15.875" x2="-6.64414375" y2="15.875" width="0.6096" layer="16"/>
 <wire x1="-6.64414375" y1="15.875" x2="-6.652621875" y2="15.866521875" width="0.6096" layer="16"/>
 <wire x1="-11.635" y1="-3.81" x2="-7.62" y2="-3.81" width="0.6096" layer="16"/>
@@
 <wire x1="-70.485" y1="23.8125" x2="-71.1725" y2="24.5" width="0.6096" layer="16"/>
 <wire x1="-71.1725" y1="24.5" x2="-71.91625" y2="24.5" width="0.6096" layer="16"/>
-<wire x1="-1.27" y1="2.54" x2="-1.27" y2="15.875" width="0.6096" layer="16"/>
 <wire x1="69.31" y1="-3.38" x2="67.105" y2="-3.38" width="0.6096" layer="16"/>
 <wire x1="67.105" y1="-3.38" x2="64.65875" y2="-5.82625" width="0.6096" layer="16"/>
@@
 <wire x1="-109.06125" y1="-22.86" x2="-105.56875" y2="-26.3525" width="0.6096" layer="16"/>
 <wire x1="-105.56875" y1="-26.3525" x2="-105.56875" y2="-29.51" width="0.6096" layer="16"/>
-<wire x1="-94.13875" y1="28.2575" x2="-94.13875" y2="29.21" width="0" layer="19" extent="16-16"/>
 <wire x1="-105.56875" y1="-29.51" x2="-103.17625" y2="-30.895" width="0.6096" layer="16"/>
+<wire x1="-13.3375" y1="10.625" x2="-12.5875" y2="12.3825" width="0.6096" layer="16"/>
+<wire x1="-6.652621875" y1="15.866521875" x2="-6.652621875" y2="14.937378125" width="0.6096" layer="16"/>
+<wire x1="-1.27" y1="2.54" x2="-1.27" y2="9.55475625" width="0.6096" layer="16"/>
+<wire x1="-1.27" y1="9.55475625" x2="-3.477621875" y2="11.762378125" width="0.6096" layer="16"/>
+<wire x1="-3.477621875" y1="11.762378125" x2="-6.652621875" y2="14.937378125" width="0.6096" layer="16"/>
+<wire x1="2.8575" y1="15.875" x2="2.2225" y2="15.24" width="0.6096" layer="16"/>
+<wire x1="2.2225" y1="15.24" x2="2.2225" y2="12.065" width="0.6096" layer="16"/>
+<wire x1="2.2225" y1="12.065" x2="1.919878125" y2="11.762378125" width="0.6096" layer="16"/>
+<wire x1="1.919878125" y1="11.762378125" x2="-3.477621875" y2="11.762378125" width="0.6096" layer="16"/>
+<wire x1="-12.5875" y1="12.3825" x2="-9.2075" y2="12.3825" width="0.6096" layer="16"/>
+<wire x1="-9.2075" y1="12.3825" x2="-6.652621875" y2="14.937378125" width="0.6096" layer="16"/>
+<wire x1="-94.13875" y1="29.21" x2="-94.13875" y2="28.2575" width="0" layer="19" extent="16-16"/>
 </signal>
 <signal name="AVCC">
@@
 <contactref element="IC4" pad="6"/>
 <contactref element="R61" pad="1"/>
-<wire x1="-21.81" y1="21.175" x2="-14.605" y2="14.2875" width="0.4064" layer="16"/>
-<wire x1="-14.605" y1="14.2875" x2="-13.65" y2="13.97" width="0.4064" layer="16"/>
+<wire x1="-21.81" y1="21.175" x2="-17.4625" y2="17.145" width="0.4064" layer="16"/>
+<wire x1="-17.4625" y1="17.145" x2="-16.1925" y2="15.8725" width="0.4064" layer="16"/>
 <wire x1="-21.81" y1="21.175" x2="-26.67" y2="23.495" width="0.4064" layer="16"/>
 <wire x1="-26.67" y1="23.495" x2="-28.515578125" y2="23.771884375" width="0.4064" layer="16"/>
@@
 <wire x1="-19.05" y1="2.5375" x2="-16.51" y2="-0.0025" width="0.4064" layer="16"/>
 <wire x1="-16.51" y1="-0.0025" x2="-14.9225" y2="-0.0025" width="0.4064" layer="16"/>
-<wire x1="-19.05" y1="2.5375" x2="-19.05" y2="10.795" width="0.4064" layer="16"/>
-<wire x1="-19.05" y1="10.795" x2="-18.415" y2="11.43" width="0.4064" layer="16"/>
-<wire x1="-18.415" y1="11.43" x2="-18.415" y2="15.875" width="0.4064" layer="16"/>
+<wire x1="-19.05" y1="2.5375" x2="-19.05" y2="11.7475" width="0.4064" layer="16"/>
+<wire x1="-19.05" y1="11.7475" x2="-18.415" y2="12.3825" width="0.4064" layer="16"/>
+<wire x1="-18.415" y1="12.3825" x2="-18.415" y2="15.875" width="0.4064" layer="16"/>
 <wire x1="-22.7625" y1="20.2225" x2="-26.9875" y2="22.225" width="0.4064" layer="16"/>
 <wire x1="-26.9875" y1="22.225" x2="-28.626265625" y2="22.506715625" width="0.4064" layer="16"/>
@@
 <contactref element="VT31" pad="C"/>
 <contactref element="R62" pad="1"/>
-<wire x1="-9.2075" y1="7.4725" x2="-13.505" y2="7.4725" width="0.4064" layer="16"/>
-<wire x1="-13.505" y1="7.4725" x2="-14.9225" y2="8.89" width="0.4064" layer="16"/>
-<wire x1="-14.9225" y1="8.89" x2="-16.8275" y2="8.89" width="0.4064" layer="16"/>
-<wire x1="-16.8275" y1="8.89" x2="-17.78" y2="7.9375" width="0.4064" layer="16"/>
-<wire x1="-17.78" y1="7.9375" x2="-17.78" y2="4.1275" width="0.4064" layer="16"/>
+<wire x1="-17.78" y1="7.62" x2="-17.78" y2="4.1275" width="0.4064" layer="16"/>
 <wire x1="-17.78" y1="4.1275" x2="-15.5575" y2="1.905" width="0.4064" layer="16"/>
 <wire x1="-15.5575" y1="1.905" x2="-14.2875" y2="1.905" width="0.4064" layer="16"/>
@@
 <wire x1="-13.335" y1="2.8575" x2="-13.335" y2="3.4925" width="0.4064" layer="16"/>
 <wire x1="-13.335" y1="3.4925" x2="-13.380125" y2="3.537625" width="0.4064" layer="16"/>
+<wire x1="-14.2875" y1="8.425" x2="-14.7525" y2="8.89" width="0.4064" layer="16"/>
+<wire x1="-14.7525" y1="8.89" x2="-16.51" y2="8.89" width="0.4064" layer="16"/>
+<wire x1="-17.78" y1="7.62" x2="-16.51" y2="8.89" width="0.4064" layer="16"/>
 </signal>
 <signal name="N$65">
@@
 <contactref element="R61" pad="2"/>
 <contactref element="VD31" pad="C"/>
-<wire x1="-10.1575" y1="9.6725" x2="-10.1575" y2="12.18" width="0.6096" layer="16"/>
-<wire x1="-10.1575" y1="12.18" x2="-9.955" y2="12.3825" width="0.6096" layer="16"/>
-<wire x1="-11.75" y1="13.97" x2="-9.955" y2="12.3825" width="0.6096" layer="16"/>
+<wire x1="-15.2375" y1="10.625" x2="-15.9875" y2="12.3825" width="0.6096" layer="16"/>
+<wire x1="-16.1925" y1="13.9725" x2="-15.9875" y2="12.3825" width="0.6096" layer="16"/>
 </signal>
 <signal name="N$66">

Commit message: e1e2
Parts:
- added R105, R111: (no value), rcl:R0805
- added R112, R114: (no value), rcl:M0805
- added RE1, RE2: (no value), pinhead:1X01
- added VD53, VD54: (no value), diode:SOD80C
- added VT53, VT54: (no value), transistor-npn:SOT23-BEC
- moved R52 9.27 mm to (-5.08, 21.6), turned to 270 degrees
- moved VD24 4.54 mm to (13.0, 9.05), turned to 90 degrees
- moved VT26 3.18 mm to (-10.5, 25.4), turned to 135 degrees
- moved VT25 1.93 mm to (10.5, 15.9)
- moved VD25 1.62 mm to (6.99, 16.5)
- moved VD30 1.35 mm to (-7.62, 19.1)
- moved VT24 1.31 mm to (17.1, 9.05)
- moved R51 1.27 mm to (-16.5, 25.1)
- moved VD26 1.14 mm to (-12.7, 27.6), turned to 135 degrees
- moved R49 1.00 mm to (8.26, 12.4)
- moved R64 0.90 mm to (-10.2, -14.0)
- moved R48 0.71 mm to (11.7, 1.91)
Connections:
- new net N$113: R114.1, VT54.C
- new net N$116: R105.2, VD54.C, VT54.B
- new net N$73: R112.1, VT53.C
- new net N$84: R111.2, VD53.C, VT53.B
- new net RE1: R111.1, RE1.1
- new net RE2: R105.1, RE2.1
- net E1: now also R112.2
- net E2: now also R114.2
- net GND: now also VD53.A, VD54.A, VT53.E, VT54.E
Routing:
- net B13: track 27.7 -> 43.2 mm
- net +100V: track 911.6 -> 925.5 mm
- net GND: track 1810.5 -> 1818.8 mm
- net N$116: track 0.00 -> 6.19 mm
- net N$84: track 0.00 -> 4.17 mm
- net N$54: track 2.71 -> 5.99 mm
- net N$51: track 22.9 -> 20.0 mm
- net RE2: track 0.00 -> 2.48 mm
- net RE1: track 0.00 -> 2.22 mm
- net E1: track 0.00 -> 2.13 mm
- net E2: track 0.00 -> 2.09 mm
- net N$113: track 0.00 -> 1.76 mm
- net N$73: track 0.00 -> 1.76 mm
- net RB13: track 14.9 -> 13.7 mm
- net N$55: track 5.46 -> 4.31 mm
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
Commit message: .
Parts:
- moved VD31 1.00 mm to (-13.3, 12.7)
- moved R61 0.45 mm to (-16.5, 14.6)
- moved VT31 0.32 mm to (-14.0, 9.53)
Routing:
- net GND: track 1818.8 -> 1817.2 mm
- net +100V: track 925.5 -> 926.0 mm
- net N$64: track 14.2 -> 13.6 mm
Changed lines of the file:
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@@
 <element name="R60" library="rcl" package="0207/12" value="" x="-9.8425" y="13.6525" rot="R315"/>
 <element name="VD30" library="diode" package="SOD80C" value="" x="-7.62" y="19.05" rot="MR270"/>
-<element name="VT31" library="transistor-npn" package="SOT23-BEC" value="" x="-14.2875" y="9.525" rot="MR180"/>
-<element name="R61" library="rcl" package="R0805" value="" x="-16.1925" y="14.9225" rot="MR270"/>
+<element name="VT31" library="transistor-npn" package="SOT23-BEC" value="" x="-13.97" y="9.525" rot="MR180"/>
+<element name="R61" library="rcl" package="R0805" value="" x="-16.51" y="14.605" rot="MR270"/>
 <element name="R62" library="rcl" package="0207/12" value="" x="-8.89" y="-0.9525" rot="R315"/>
-<element name="VD31" library="diode" package="SOD80C" value="" x="-14.2875" y="12.3825" rot="MR180"/>
+<element name="VD31" library="diode" package="SOD80C" value="" x="-13.335" y="12.7" rot="MR180"/>
 <element name="VT32" library="transistor-npn" package="SOT23-BEC" value="" x="-13.97" y="-6.985" rot="MR180"/>
 <element name="R63" library="rcl" package="R0805" value="" x="-14.9225" y="-0.9525" rot="MR270"/>
@@
 <wire x1="-105.56875" y1="-26.3525" x2="-105.56875" y2="-29.51" width="0.6096" layer="16"/>
 <wire x1="-105.56875" y1="-29.51" x2="-103.17625" y2="-30.895" width="0.6096" layer="16"/>
-<wire x1="-13.3375" y1="10.625" x2="-12.5875" y2="12.3825" width="0.6096" layer="16"/>
+<wire x1="-13.02" y1="10.625" x2="-11.635" y2="12.7" width="0.6096" layer="16"/>
 <wire x1="-1.27" y1="2.54" x2="-1.27" y2="9.55475625" width="0.6096" layer="16"/>
-<wire x1="-1.27" y1="9.55475625" x2="-3.477621875" y2="11.762378125" width="0.6096" layer="16"/>
+<wire x1="-1.27" y1="9.55475625" x2="-1.255121875" y2="11.762378125" width="0.6096" layer="16"/>
 <wire x1="2.2225" y1="14.9225" x2="2.2225" y2="12.065" width="0.6096" layer="16"/>
 <wire x1="2.2225" y1="12.065" x2="1.919878125" y2="11.762378125" width="0.6096" layer="16"/>
-<wire x1="1.919878125" y1="11.762378125" x2="-3.477621875" y2="11.762378125" width="0.6096" layer="16"/>
-<wire x1="-12.5875" y1="12.3825" x2="-9.8425" y2="12.3825" width="0.6096" layer="16"/>
-<wire x1="-9.8425" y1="12.3825" x2="-9.2075" y2="12.3825" width="0.6096" layer="16"/>
-<wire x1="-3.477621875" y1="11.762378125" x2="-8.587378125" y2="11.762378125" width="0.6096" layer="16"/>
-<wire x1="-8.587378125" y1="11.762378125" x2="-9.2075" y2="12.3825" width="0.6096" layer="16"/>
-<wire x1="-10.0125" y1="17.1475" x2="-10.0125" y2="12.5525" width="0.6096" layer="16"/>
-<wire x1="-10.0125" y1="12.5525" x2="-9.8425" y2="12.3825" width="0.6096" layer="16"/>
+<wire x1="1.919878125" y1="11.762378125" x2="-1.255121875" y2="11.762378125" width="0.6096" layer="16"/>
+<wire x1="-11.635" y1="12.7" x2="-9.8425" y2="12.7" width="0.6096" layer="16"/>
+<wire x1="-1.255121875" y1="11.762378125" x2="-8.587378125" y2="11.762378125" width="0.6096" layer="16"/>
+<wire x1="-8.587378125" y1="11.762378125" x2="-9.8425" y2="12.7" width="0.6096" layer="16"/>
+<wire x1="-10.0125" y1="17.1475" x2="-10.0125" y2="12.87" width="0.6096" layer="16"/>
+<wire x1="-10.0125" y1="12.87" x2="-9.8425" y2="12.7" width="0.6096" layer="16"/>
 <wire x1="-7.62" y1="17.35" x2="-10.0125" y2="17.1475" width="0.6096" layer="16"/>
 <contactref element="VT53" pad="E"/>
@@
 <wire x1="26.3525" y1="16.8275" x2="12.065" y2="14.9225" width="0.254" layer="1"/>
 <wire x1="12.065" y1="14.9225" x2="8.255" y2="11.1125" width="0.254" layer="1"/>
-<wire x1="8.255" y1="11.1125" x2="-16.1925" y2="11.1125" width="0.254" layer="1"/>
 <wire x1="24.765" y1="14.6025" x2="26.3525" y2="16.8275" width="0.6096" layer="16"/>
 <wire x1="93.98" y1="13.59125" x2="93.98" y2="12.7" width="0.6096" layer="16"/>
@@
 <contactref element="R109" pad="2"/>
 <wire x1="33.655" y1="-24.7625" x2="33.655" y2="-24.765" width="0.4064" layer="16"/>
+<wire x1="8.255" y1="11.1125" x2="-16.1925" y2="11.1125" width="0.254" layer="1"/>
 </signal>
 <signal name="SDA">
@@
 <contactref element="R61" pad="1"/>
 <wire x1="-21.81" y1="21.175" x2="-17.4625" y2="17.145" width="0.4064" layer="16"/>
-<wire x1="-17.4625" y1="17.145" x2="-16.1925" y2="15.8725" width="0.4064" layer="16"/>
+<wire x1="-17.4625" y1="17.145" x2="-16.51" y2="15.555" width="0.4064" layer="16"/>
 <wire x1="-21.81" y1="21.175" x2="-26.67" y2="23.495" width="0.4064" layer="16"/>
 <wire x1="-26.67" y1="23.495" x2="-28.515578125" y2="23.771884375" width="0.4064" layer="16"/>
@@
 <wire x1="-14.2875" y1="38.1" x2="-6.985" y2="30.7975" width="0.6096" layer="16"/>
 <contactref element="R78" pad="2"/>
-<wire x1="-15.56684375" y1="5.40684375" x2="-10.65190625" y2="5.40684375" width="0.6096" layer="16"/>
-<wire x1="-10.65190625" y1="5.40684375" x2="-6.808821875" y2="1.563759375" width="0.6096" layer="16"/>
+<wire x1="-11.5950625" y1="6.35" x2="-6.808821875" y2="1.563759375" width="0.6096" layer="16"/>
 <wire x1="-6.808821875" y1="1.563759375" x2="-6.1975625" y2="0.9525" width="0.6096" layer="16"/>
 <wire x1="-6.1975625" y1="0.9525" x2="-6.0325" y2="0.635" width="0.6096" layer="16"/>
@@
 <wire x1="0.149934375" y1="-14.605" x2="-1.905003125" y2="-14.605" width="0.6096" layer="16"/>
 <wire x1="-1.905003125" y1="-14.605" x2="-3.24996875" y2="-15.949965625" width="0.6096" layer="16"/>
+<wire x1="-11.5950625" y1="6.35" x2="-13.0175" y2="6.35" width="0.6096" layer="16"/>
+<wire x1="-13.0175" y1="6.35" x2="-15.56684375" y2="5.40684375" width="0.6096" layer="16"/>
 </signal>
 <signal name="E1">
@@
 <contactref element="VT31" pad="C"/>
 <contactref element="R62" pad="1"/>
-<wire x1="-17.78" y1="7.62" x2="-17.78" y2="4.1275" width="0.4064" layer="16"/>
-<wire x1="-17.78" y1="4.1275" x2="-15.5575" y2="1.905" width="0.4064" layer="16"/>
-<wire x1="-15.5575" y1="1.905" x2="-14.2875" y2="1.905" width="0.4064" layer="16"/>
-<wire x1="-14.2875" y1="1.905" x2="-13.335" y2="2.8575" width="0.4064" layer="16"/>
-<wire x1="-13.335" y1="2.8575" x2="-13.335" y2="3.4925" width="0.4064" layer="16"/>
-<wire x1="-13.335" y1="3.4925" x2="-13.380125" y2="3.537625" width="0.4064" layer="16"/>
-<wire x1="-14.2875" y1="8.425" x2="-14.7525" y2="8.89" width="0.4064" layer="16"/>
-<wire x1="-14.7525" y1="8.89" x2="-16.51" y2="8.89" width="0.4064" layer="16"/>
-<wire x1="-17.78" y1="7.62" x2="-16.51" y2="8.89" width="0.4064" layer="16"/>
+<wire x1="-17.78" y1="7.3025" x2="-17.78" y2="4.1275" width="0.4064" layer="16"/>
+<wire x1="-17.78" y1="4.1275" x2="-15.875" y2="2.2225" width="0.4064" layer="16"/>
+<wire x1="-15.875" y1="2.2225" x2="-13.97" y2="2.2225" width="0.4064" layer="16"/>
+<wire x1="-17.78" y1="7.3025" x2="-16.6575" y2="8.425" width="0.4064" layer="16"/>
+<wire x1="-16.6575" y1="8.425" x2="-13.97" y2="8.425" width="0.4064" layer="16"/>
+<wire x1="-13.97" y1="2.2225" x2="-13.380125" y2="2.812375" width="0.4064" layer="16"/>
+<wire x1="-13.380125" y1="2.812375" x2="-13.380125" y2="3.537625" width="0.4064" layer="16"/>
 </signal>
 <signal name="N$65">
@@
 <contactref element="R61" pad="2"/>
 <contactref element="VD31" pad="C"/>
-<wire x1="-15.2375" y1="10.625" x2="-15.9875" y2="12.3825" width="0.6096" layer="16"/>
-<wire x1="-16.1925" y1="13.9725" x2="-15.9875" y2="12.3825" width="0.6096" layer="16"/>
+<wire x1="-14.92" y1="10.625" x2="-15.035" y2="12.7" width="0.6096" layer="16"/>
+<wire x1="-16.51" y1="13.655" x2="-15.035" y2="12.7" width="0.6096" layer="16"/>
 </signal>
 <signal name="N$66">

Commit message: .
Parts:
- N27: value IN-3 -> IN-33; device in3:IN-3 -> in3-mod:IN-3-3
Routing:
- net E1: track 2.13 -> 0.00 mm
Changed lines of the file:
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@@
 <wire x1="116.84" y1="47.9425" x2="116.84" y2="-48.26" width="0.254" layer="20"/>
 <dimension x1="-116.84" y1="49.53" x2="116.84" y2="51.1175" x3="0" y3="53.34" textsize="1.778" layer="47" dtype="horizontal"/>
-<dimension x1="-116.84" y1="57.15" x2="0" y2="-60.96" x3="-58.42" y3="66.9925" textsize="1.778" layer="47" dtype="horizontal"/>
-<dimension x1="0" y1="70.8025" x2="116.84" y2="57.15" x3="58.42" y3="76.5175" textsize="1.778" layer="47" dtype="horizontal"/>
+<dimension x1="-31.115" y1="-57.15" x2="-17.145" y2="-67.6275" x3="-24.13" y3="66.9925" textsize="1.778" layer="47" dtype="horizontal"/>
+<dimension x1="0" y1="70.8025" x2="17.145" y2="-57.785" x3="8.5725" y3="76.5175" textsize="1.778" layer="47" dtype="horizontal"/>
 <circle x="-94.615" y="29.5275" radius="1.851325" width="0.4064" layer="209"/>
 </plain>
@@
 <element name="N25" library="in3-mod" package="IN-3-1" value="IN-31" x="-45" y="14" locked="yes" rot="R225"/>
 <element name="N26" library="in3" package="IN-3" value="IN-3" x="-31" y="0" locked="yes" rot="R180"/>
-<element name="N27" library="in3" package="IN-3" value="IN-3" x="0" y="14" locked="yes"/>
+<element name="N27" library="in3-mod" package="IN-3-3" value="IN-33" x="0" y="14" locked="yes"/>
 <element name="N28" library="in3" package="IN-3" value="IN-3" x="0" y="-14" locked="yes"/>
 <element name="N29" library="in3" package="IN-3" value="IN-3" x="17" y="28" locked="yes" rot="R135"/>
@@
 <wire x1="29.845" y1="9.2075" x2="27.6225" y2="11.43" width="0.4064" layer="16"/>
 <wire x1="27.6225" y1="11.43" x2="25.75535" y2="11.43" width="0.4064" layer="16"/>
-<wire x1="16.98625" y1="-17.2575" x2="16.98625" y2="-11.1125" width="0.6096" layer="16"/>
-<wire x1="16.98625" y1="-11.1125" x2="18.57375" y2="-9.525" width="0.6096" layer="16"/>
-<wire x1="18.57375" y1="-9.525" x2="18.57375" y2="-7.475" width="0.6096" layer="16"/>
+<wire x1="16.98625" y1="-17.2575" x2="16.98625" y2="-16.1925" width="0.6096" layer="16"/>
+<wire x1="16.98625" y1="-16.1925" x2="18.57375" y2="-14.605" width="0.6096" layer="16"/>
+<wire x1="18.57375" y1="-14.605" x2="18.57375" y2="-7.475" width="0.6096" layer="16"/>
 <wire x1="18.57375" y1="-7.475" x2="17.7775" y2="-6.36125" width="0.6096" layer="16"/>
 <wire x1="17.73375" y1="-4.28625" x2="17.7775" y2="-6.36125" width="0.6096" layer="16"/>
@@
 <contactref element="N27" pad="K"/>
 <contactref element="R112" pad="2"/>
-<wire x1="1.585" y1="-4.1275" x2="1.5875" y2="-2" width="0.6096" layer="16"/>
+<wire x1="1.585" y1="-4.1275" x2="3.5875" y2="-2" width="0" layer="19" extent="16-16"/>
 </signal>
 <signal name="E2">
