File: EAGLE/IN3-PCB/in3watch.brd (EAGLE design)
At the start: 61.9 x 90.5 mm, 132 parts, among them J3 J5MM

Commit message: .
Parts:
- moved R105 19.8 mm to (-1.59, 22.5), turned to 270 degrees
- moved R52 18.5 mm to (-7.62, 39.4)
- moved Z1 16.4 mm to (67.6, -1.91)
- moved R111 15.5 mm to (0.32, 22.5), turned to 270 degrees
- moved VT26 12.1 mm to (-10.5, 38.7)
- moved XO1 4.18 mm to (66.7, -63.5)
- moved RE1 3.19 mm to (-1.59, 28.9), turned to 180 degrees
- moved RE2 2.03 mm to (-1.59, 26.4), turned to 0 degrees
- moved VT53 0.32 mm to (-0.64, -8.57)
Routing:
- net N$116: track 2.83 -> 48.9 mm, vias 0 -> 2
- net N$84: track 0.00 -> 29.4 mm, vias 0 -> 1
- net +100V: track 237.6 -> 266.5 mm
- net RE1: track 0.00 -> 6.93 mm
- net RE2: track 0.00 -> 2.86 mm
Other:
- board size 61.9 x 90.5 mm -> 61.9 x 89.9 mm

Commit message: .
Parts:
- added DD1B1: DS1307/PCF8583, ds1307_pcf8583:SO8-7_5+SOIC8
- moved DD1B 127.6 mm to (-30.6, 64.4), turned to 0 degrees
- moved J3 126.2 mm to (-41.6, 49.4)
- moved Z1 77.5 mm to (0.64, 37.1), turned to 90 degrees
- moved XN1 68.6 mm to (56.2, -26.4)
- moved R108 63.1 mm to (80.8, 50.5)
- moved R107 60.9 mm to (78.2, 46.4)
- moved J4 58.6 mm to (83.7, 39.2)
- moved DD2 50.8 mm to (89.3, 30.2), flipped to the bottom, turned to 90 degrees
- moved C5 26.0 mm to (78.9, 14.6)
- moved DD1A 9.86 mm to (85.2, -3.17)
- moved XN4 2.31 mm to (134.3, -80.6)
Connections:
- new net VCC: DD1B1.8
- net GND: now also DD1B1.4
Other:
- board text added: "IP/2"

Commit message: .
Parts:
- removed DATAIN: (no value), Разъёмы штырьковые 2.54мм:1X03
- removed QO1, QO2: (no value), Разъёмы штырьковые 2.54мм:1X01
- added JP2: (no value), Разъёмы штырьковые 2.54мм:1X05
- moved C12 72.6 mm to (44.5, -56.2)
- moved C9 66.1 mm to (35.9, -51.4)
- moved C13 60.4 mm to (40.3, -55.6)
- moved C10 59.3 mm to (35.2, -54.9)
- moved C11 58.2 mm to (40.3, -51.8)
- moved J5 30.3 mm to (121.9, 5.08)
- moved VD53 21.0 mm to (0.64, 9.21), turned to 180 degrees
- moved VT53 14.0 mm to (0.00, 5.40), turned to 180 degrees
- moved J3 11.3 mm to (-30.5, 51.3)
- moved R112 6.70 mm to (0.95, 1.59), turned to 270 degrees
- moved C2 1.27 mm to (20.0, -75.6)
- moved C1 1.27 mm to (18.4, -61.9), turned to 90 degrees
- moved JP4 0.32 mm to (13.7, -78.4)
Connections:
- net RCLOCK: now also JP2.3; no longer DATAIN.1
- net RLATCH: now also JP2.2; no longer DATAIN.2
- net SER0: now also JP2.1; no longer DATAIN.3
- net SER1: now also JP2.4; no longer QO1.1
- net SER2: now also JP2.5; no longer QO2.1
Routing:
- net GND: track 158.6 -> 218.9 mm, vias 11 -> 14
- net N$84: track 29.4 -> 15.7 mm, vias 1 -> 0
- net +5V: track 150.1 -> 163.1 mm
- net SER2: track 39.9 -> 52.5 mm
- net R7: track 44.1 -> 49.4 mm
- net N$116: track 48.9 -> 45.6 mm, vias 2 -> 0
- net RLATCH: track 99.9 -> 102.0 mm
- net R1: track 80.5 -> 82.2 mm, vias 5 -> 7
- net RCLOCK: track 95.5 -> 96.9 mm
- net SER1: track 33.3 -> 34.4 mm
- net +100V: track 266.5 -> 267.4 mm
- net N$73: track 2.71 -> 2.00 mm
- net E1: track 2.13 -> 2.71 mm
