File: EAGLE/IN3-PCB/in3watch.sch (EAGLE design)
At the start: 312 parts, among them IC1 74HC595D, IC2 74HC595D, IC3 74HC595D, IC4 74HC595D, IC5 74HC595D, IC6 74HC595D, IC7 74HC595D, J3 J5MM

Commit message: .
Parts:
- removed IC1, IC2, IC3, IC4, IC5, IC6, IC7: 74HC595D, 74xx-eu:74HC595D
- removed J6, R19, R75: (no value), rcl:R-EU_R1206W
- removed N1, N10, N11, N12, N13, N15, N16, N17, N18, N19, N2, N20, N21, N22, N26, N43, N44, N45, N46, N47, N48, N49, N50, N54, N7, N8, N9: IN-3, in3:IN-3
- removed N14, N23, N24, N25, N42, N51: IN-31, in3-mod:IN-31
- removed N3, N4, N5, N6: IN-32, in3-mod:IN-32
- removed N52, N53: IN-311, in3-mod:IN-311
- removed R1, R101, R103, R11, R13, R15, R17, R21, R23, R25, R3, R5, R53, R55, R57, R59, R61, R63, R65, R67, R69, R7, R71, R73, R77, R79, R81, R83, R85, R87, R89, R9, R93, R95, R97, R99: (no value), rcl:R-EU_R0805
- removed R10, R100, R102, R12, R14, R16, R18, R2, R20, R22, R24, R26, R4, R54, R58, R6, R60, R62, R64, R66, R68, R70, R72, R74, R8, R80, R82, R84, R86, R88, R90, R91, R92, R94, R96, R98: (no value), rcl:R-EU_0207/12
- removed R104, R78: (no value), rcl:R-EU_0207/15
- removed R56, R76: (no value), rcl:R-EU_0207/10
- removed VD1, VD10, VD11, VD12, VD13, VD2, VD27, VD28, VD29, VD3, VD30, VD31, VD32, VD33, VD34, VD35, VD36, VD37, VD38, VD39, VD4, VD40, VD41, VD42, VD43, VD44, VD45, VD46, VD47, VD48, VD49, VD5, VD50, VD51, VD52, VD6, VD7, VD8, VD9: (no value), diode:ZENER-DIODESOD80C
- removed VT1, VT10, VT11, VT12, VT13, VT2, VT27, VT28, VT29, VT3, VT30, VT31, VT32, VT33, VT34, VT35, VT36, VT37, VT38, VT39, VT4, VT40, VT41, VT42, VT43, VT44, VT45, VT46, VT47, VT48, VT49, VT5, VT50, VT51, VT52, VT6, VT7, VT8, VT9: BC849SMD, transistor-npn:BC849SMD
- added DATAIN, XI2, XO1: (no value), Разъёмы штырьковые 2.54мм:PINHD-1X3
- added DDD1, DDD2, DDD3, DDD4, DDD5, DDD6, DDD7: 74HC595D, 74xx-eu:74HC595D
- added JP4: (no value), Разъёмы штырьковые 2.54мм:PINHD-1X2
- added JS1: (no value), jumper:SJ2W
- added QO1, QO2, XO3: (no value), Разъёмы штырьковые 2.54мм:PINHD-1X1
- added XI2B, XO2B: (no value), Разъёмы штырьковые 2.54мм:PINHD-1X2/2
- added XN1, XN2, XN3, XN4: (no value), Разъёмы штырьковые 2.54мм:PINHD-1X13
- added XO2A: (no value), Разъёмы штырьковые 2.54мм:PINHD-1X6
- added XO4: (no value), Разъёмы штырьковые 2.54мм:PINHD-1X4
- N27: value IN-33 -> IN-3; device in3-mod:IN-33 -> in3:IN-3
Connections:
- removed net A1: N42.K, R2.2
- removed net A10: N51.K, R20.2
- removed net A11: N52.K, R22.2
- removed net A12: N53.K, R24.2
- removed net A13: N54.K, R26.2
- removed net A2: N43.K, R4.2
- removed net A3: N44.K, R6.2
- removed net A4: N45.K, R8.2
- removed net A5: N46.K, R10.2
- removed net A6: N47.K, R12.2
- removed net A7: N48.K, R14.2
- removed net A8: N49.K, R16.2
- removed net A9: N50.K, R18.2
- removed net C1: N14.K, R54.2
- removed net C10: N23.K, R72.2
- removed net C11: N24.K, R74.2
- removed net C12: N25.K, R76.2
- removed net C13: N26.K, VT39.C
- removed net C2: N15.K, R56.2
- removed net C3: N16.K, R58.2
- removed net C4: N17.K, R60.2
- removed net C5: N18.K, R62.2
- removed net C6: N19.K, R64.2
- removed net C7: N20.K, R66.2
- removed net C8: N21.K, R68.2
- removed net C9: N22.K, R70.2
- removed net D1: N1.K, R80.2
- removed net D10: N10.K, R98.2
- removed net D11: N11.K, R100.2
- removed net D12: N12.K, R102.2
- removed net D13: N13.K, R104.2
- removed net D2: N2.K, R82.2
- removed net D3: N3.K, R84.2
- removed net D4: N4.K, R86.2
- removed net D5: N5.K, R88.2
- removed net D6: N6.K, R90.2
- removed net D7: N7.K, R92.2
- removed net D8: N8.K, R94.2
- removed net D9: N9.K, R96.2
- removed net N$1: R2.1, VT1.C
- removed net N$10: R22.1, VT11.C
- removed net N$100: R94.1, VT47.C
- removed net N$101: R93.2, VD47.C, VT47.B
- removed net N$102: R96.1, VT48.C
- removed net N$103: R95.2, VD48.C, VT48.B
- removed net N$104: R98.1, VT49.C
- removed net N$105: R97.2, VD49.C, VT49.B
- removed net N$106: R100.1, VT50.C
- removed net N$107: R99.2, VD50.C, VT50.B
- removed net N$108: R102.1, VT51.C
- removed net N$109: R101.2, VD51.C, VT51.B
- removed net N$11: R21.2, VD11.C, VT11.B
- removed net N$110: R104.1, VT52.C
- removed net N$111: R103.2, VD52.C, VT52.B
- removed net N$12: R24.1, VT12.C
- removed net N$13: R23.2, VD12.C, VT12.B
- removed net N$14: R26.1, VT13.C
- removed net N$15: R25.2, VD13.C, VT13.B
- removed net N$18: R6.1, VT3.C
- removed net N$19: R5.2, VD3.C, VT3.B
- removed net N$2: R1.2, VD1.C, VT1.B
- removed net N$20: R8.1, VT4.C
- removed net N$21: R7.2, VD4.C, VT4.B
- removed net N$22: R10.1, VT5.C
- removed net N$23: R9.2, VD5.C, VT5.B
- removed net N$24: R12.1, VT6.C
- removed net N$25: R11.2, VD6.C, VT6.B
- removed net N$26: R14.1, VT7.C
- removed net N$27: R13.2, VD7.C, VT7.B
- removed net N$28: R16.1, VT8.C
- removed net N$29: R15.2, VD8.C, VT8.B
- removed net N$4: R4.1, VT2.C
- removed net N$5: R3.2, VD2.C, VT2.B
- removed net N$56: R54.1, VT27.C
- removed net N$57: R53.2, VD27.C, VT27.B
- removed net N$58: R56.1, VT28.C
- removed net N$59: R55.2, VD28.C, VT28.B
- removed net N$6: R18.1, VT9.C
- removed net N$60: R58.1, VT29.C
- removed net N$61: R57.2, VD29.C, VT29.B
- removed net N$62: R60.1, VT30.C
- removed net N$63: R59.2, VD30.C, VT30.B
- removed net N$64: R62.1, VT31.C
- removed net N$65: R61.2, VD31.C, VT31.B
- removed net N$66: R64.1, VT32.C
- removed net N$67: R63.2, VD32.C, VT32.B
- removed net N$68: R66.1, VT33.C
- removed net N$69: R65.2, VD33.C, VT33.B
- removed net N$7: R17.2, VD9.C, VT9.B
- removed net N$70: R68.1, VT34.C
- removed net N$71: R67.2, VD34.C, VT34.B
- removed net N$74: R70.1, VT35.C
- removed net N$75: R69.2, VD35.C, VT35.B
- removed net N$77: N26.A, R78.1
- removed net N$78: R72.1, VT36.C
- removed net N$79: R71.2, VD36.C, VT36.B
- removed net N$8: R20.1, VT10.C
- removed net N$80: R74.1, VT37.C
- removed net N$81: R73.2, VD37.C, VT37.B
- removed net N$82: R76.1, VT38.C
- removed net N$83: R75.2, VD38.C, VT38.B
- removed net N$85: R77.2, VD39.C, VT39.B
- removed net N$86: R80.1, VT40.C
- removed net N$87: R79.2, VD40.C, VT40.B
- removed net N$88: R82.1, VT41.C
- removed net N$89: R81.2, VD41.C, VT41.B
- removed net N$9: R19.2, VD10.C, VT10.B
- removed net N$90: R84.1, VT42.C
- removed net N$91: R83.2, VD42.C, VT42.B
- removed net N$92: R86.1, VT43.C
- removed net N$93: R85.2, VD43.C, VT43.B
- removed net N$94: R88.1, VT44.C
- removed net N$95: R87.2, VD44.C, VT44.B
- removed net N$96: R90.1, VT45.C
- removed net N$97: R89.2, VD45.C, VT45.B
- removed net N$98: R92.1, VT46.C
- removed net N$99: R91.2, VD46.C, VT46.B
- removed net RA1: IC1A.QA, R1.1
- removed net RA10: IC2A.QB, R19.1
- removed net RA11: IC2A.QC, R21.1
- removed net RA12: IC2A.QD, R23.1
- removed net RA13: IC2A.QE, R25.1
- removed net RA2: IC1A.QB, R3.1
- removed net RA3: IC1A.QC, R5.1
- removed net RA4: IC1A.QD, R7.1
- removed net RA5: IC1A.QE, R9.1
- removed net RA6: IC1A.QF, R11.1
- removed net RA7: IC1A.QG, R13.1
- removed net RA8: IC1A.QH, R15.1
- removed net RA9: IC2A.QA, R17.1
- removed net RC1: IC4A.QC, R53.1
- removed net RC10: IC5A.QD, R71.1
- removed net RC11: IC5A.QE, R73.1
- removed net RC12: IC5A.QF, R75.1
- removed net RC13: IC5A.QG, R77.1
- removed net RC2: IC4A.QD, R55.1
- removed net RC3: IC4A.QE, R57.1
- removed net RC4: IC4A.QF, R59.1
- removed net RC5: IC4A.QG, R61.1
- removed net RC6: IC4A.QH, R63.1
- removed net RC7: IC5A.QA, R65.1
- removed net RC8: IC5A.QB, R67.1
- removed net RC9: IC5A.QC, R69.1
- removed net RD1: IC5A.QH, R79.1
- removed net RD10: IC7A.QA, R97.1
- removed net RD11: IC7A.QB, R99.1
- removed net RD12: IC7A.QC, R101.1
- removed net RD13: IC7A.QD, R103.1
- removed net RD2: IC6A.QA, R81.1
- removed net RD3: IC6A.QB, R83.1
- removed net RD4: IC6A.QC, R85.1
- removed net RD5: IC6A.QD, R87.1
- removed net RD6: IC6A.QE, R89.1
- removed net RD7: IC6A.QF, R91.1
- removed net RD8: IC6A.QG, R93.1
- removed net RD9: IC6A.QH, R95.1
- removed net SER3: IC2A.QH*, IC3A.SER
- removed net SER4: IC3A.QH*, IC4A.SER
- removed net SER5: IC4A.QH*, J6.1
- removed net SER6: IC5A.QH*, IC6A.SER
- removed net SER7: IC6A.QH*, IC7A.SER
- new net N$117: DDD7A.QF, XO4.2
- new net N$118: DDD7A.QG, XO4.3
- new net N$119: DDD7A.QH, XO4.4
- new net R1: DDD1A.QA, DDD2A.QF, DDD4A.QC, DDD5A.QH, XI2.1, XN1.1, XN2.1, XN3.1, XN4.1, XO1.1, XO2A.1, XO3.1
- new net R10: DDD2A.QB, DDD3A.QG, DDD5A.QD, DDD7A.QA, XN1.10, XN2.10, XN3.10, XN4.10
- new net R11: DDD2A.QC, DDD3A.QH, DDD5A.QE, DDD7A.QB, XN1.11, XN2.11, XN3.11, XN4.11
- new net R12: DDD2A.QD, DDD4A.QA, DDD5A.QF, DDD7A.QC, XI2B.1, XN1.12, XN2.12, XN3.12, XN4.12, XO2B.1
- new net R13: DDD2A.QE, DDD4A.QB, DDD5A.QG, DDD7A.QD, XI2B.2, XN1.13, XN2.13, XN3.13, XN4.13, XO2B.2
- new net R2: DDD1A.QB, DDD2A.QG, DDD4A.QD, DDD6A.QA, XI2.2, XN1.2, XN2.2, XN3.2, XN4.2, XO1.2, XO2A.2
- new net R3: DDD1A.QC, DDD2A.QH, DDD4A.QE, DDD6A.QB, XI2.3, XN1.3, XN2.3, XN3.3, XN4.3, XO1.3, XO2A.3
- new net R4: DDD1A.QD, DDD3A.QA, DDD4A.QF, DDD6A.QC, XN1.4, XN2.4, XN3.4, XN4.4, XO2A.4
- new net R5: DDD1A.QE, DDD3A.QB, DDD4A.QG, DDD6A.QD, XN1.5, XN2.5, XN3.5, XN4.5, XO2A.5
- new net R6: DDD1A.QF, DDD3A.QC, DDD4A.QH, DDD6A.QE, XN1.6, XN2.6, XN3.6, XN4.6, XO2A.6
- new net R7: DDD1A.QG, DDD3A.QD, DDD5A.QA, DDD6A.QF, XN1.7, XN2.7, XN3.7, XN4.7
- new net R8: DDD1A.QH, DDD3A.QE, DDD5A.QB, DDD6A.QG, XN1.8, XN2.8, XN3.8, XN4.8
- new net R9: DDD2A.QA, DDD3A.QF, DDD5A.QC, DDD6A.QH, XN1.9, XN2.9, XN3.9, XN4.9
- new net RCLOCK: DATAIN.1, DDD1A.SCK, DDD2A.SCK, DDD3A.SCK, DDD4A.SCK, DDD5A.SCK, DDD6A.SCK, DDD7A.SCK
- new net RDATA: DDD5A.SER
- new net RLATCH: DATAIN.2, DDD1A.RCK, DDD2A.RCK, DDD3A.RCK, DDD4A.RCK, DDD5A.RCK, DDD6A.RCK, DDD7A.RCK
- new net SER0: DATAIN.3, DDD1A.SER, DDD3A.SER, DDD6A.SER
- new net SER1: DDD1A.QH*, DDD2A.SER, DDD3A.QH*, DDD4A.SER, DDD6A.QH*, DDD7A.SER, QO1.1
- net +100V: no longer N1.A, N10.A, N11.A, N12.A, N13.A, N14.A, N15.A, N16.A, N17.A, N18.A, N19.A, N2.A, N20.A, N21.A, N22.A, N23.A, N24.A, N25.A, N3.A, N4.A, N42.A, N43.A, N44.A, N45.A, N46.A, N47.A, N48.A, N49.A, N5.A, N50.A, N51.A, N52.A, N53.A, N54.A, N6.A, N7.A, N8.A, N9.A, R78.2
- net +5V: now also DDD1A.SCL, DDD1P.VCC, DDD2A.SCL, DDD2P.VCC, DDD3A.SCL, DDD3P.VCC, DDD4A.SCL, DDD4P.VCC, DDD5A.SCL, DDD5P.VCC, DDD6A.SCL, DDD6P.VCC, DDD7A.SCL, DDD7P.VCC, JP4.1; no longer IC1A.SCL, IC1P.VCC, IC2A.SCL, IC2P.VCC, IC3A.SCL, IC3P.VCC, IC4A.SCL, IC4P.VCC, IC5A.SCL, IC5P.VCC, IC6A.SCL, IC6P.VCC, IC7A.SCL, IC7P.VCC
- net B13: no longer R52.2
- net GND: now also DDD1A.G, DDD1P.GND, DDD2A.G, DDD2P.GND, DDD3A.G, DDD3P.GND, DDD4A.G, DDD4P.GND, DDD5A.G, DDD5P.GND, DDD6A.G, DDD6P.GND, DDD7A.G, DDD7P.GND, JP4.2; no longer IC1A.G, IC1P.GND, IC2A.G, IC2P.GND, IC3A.G, IC3P.GND, IC4A.G, IC4P.GND, IC5A.G, IC5P.GND, IC6A.G, IC6P.GND, IC7A.G, IC7P.GND, VD1.A, VD10.A, VD11.A, VD12.A, VD13.A, VD2.A, VD27.A, VD28.A, VD29.A, VD3.A, VD30.A, VD31.A, VD32.A, VD33.A, VD34.A, VD35.A, VD36.A, VD37.A, VD38.A, VD39.A, VD4.A, VD40.A, VD41.A, VD42.A, VD43.A, VD44.A, VD45.A, VD46.A, VD47.A, VD48.A, VD49.A, VD5.A, VD50.A, VD51.A, VD52.A, VD6.A, VD7.A, VD8.A, VD9.A, VT1.E, VT10.E, VT11.E, VT12.E, VT13.E, VT2.E, VT27.E, VT28.E, VT29.E, VT3.E, VT30.E, VT31.E, VT32.E, VT33.E, VT34.E, VT35.E, VT36.E, VT37.E, VT38.E, VT39.E, VT4.E, VT40.E, VT41.E, VT42.E, VT43.E, VT44.E, VT45.E, VT46.E, VT47.E, VT48.E, VT49.E, VT5.E, VT50.E, VT51.E, VT52.E, VT6.E, VT7.E, VT8.E, VT9.E
- net N$17: now also DDD7A.QE, XO4.1; no longer IC5A.SER, J6.2
- net RB1: no longer IC2A.QF
- net RB10: no longer IC3A.QG
- net RB11: no longer IC3A.QH
- net RB12: no longer IC4A.QA
- net RB13: no longer IC4A.QB
- net RB2: no longer IC2A.QG
- net RB3: no longer IC2A.QH
- net RB4: no longer IC3A.QA
- net RB5: no longer IC3A.QB
- net RB6: no longer IC3A.QC
- net RB7: no longer IC3A.QD
- net RB8: no longer IC3A.QE
- net RB9: no longer IC3A.QF
- net RCLOCK_MISO_D12: no longer IC1A.SCK, IC2A.SCK, IC3A.SCK, IC4A.SCK, IC5A.SCK, IC6A.SCK, IC7A.SCK
- net RDATA_MOSI_D11: no longer IC1A.SER
- net RLATCH_D10: no longer IC1A.RCK, IC2A.RCK, IC3A.RCK, IC4A.RCK, IC5A.RCK, IC6A.RCK, IC7A.RCK
- net SER2: now also DDD2A.QH*, DDD4A.QH*, DDD5A.QH*, DDD7A.QH*, QO2.1; no longer IC1A.QH*, IC2A.SER
Other:
- note added: "1 ic1 ic2 2 ic3 3 ic4 ic5 4 ic6 ic7"
- note added: "RA1 RA2 RA3 RA4 RA5 RA6 RA7 RA8"
- note added: "RA1 RA2 RA3 RA4 RA5 RA6 RA7 RA8 RA9 RA10 RA11 RA12 RA13"
- note added: "RA9 RA10 RA11 RA12 RA13 RB1 RB2 RB3"
- note added: "RB1 RB2 RB3"
- note added: "RB12 RB13"
- note added: "RB12 RB13 RС1 RС2 RС3 RС4 RС5 RС6"
- note added: "RB4 RB5 RB6 RB7 RB8"
- note added: "RB4 RB5 RB6 RB7 RB8 RB9 RB10 RB11"
- note added: "RC7 RC8 RC9 RC10 RC11 RC12 RC13 RD1"
- note added: "RD10 RD11 RD12 RD13"
- note added: "RD2 RD3 RD4 RD5 RD6 RD7 RD8 RD9"
- note added: "RС1 RС2 RС3 RС4 RС5 RС6"
- note added: "RС1 RС2 RС3 RС4 RС5 RС6 RC7 RC8 RC9 RC10 RC11 RC12 RC13"
- note added: "SEGMENT_1 DDD1 DDD2 OR SEGMENT_2 (DDD1 DDD2) DDD3 DDD4 SER0=in SER2=QO2=out - SEGMENT_2+ (DDD1 DDD2) DDD3 SER0=in SER1=QO1=out"
- note added: "SEGMENT_3 DDD4 DDD5 SER1=in SER2=QO2=out"

Commit message: .
Parts:
- added DD1B1: DS1307/PCF8583, ds1307_pcf8583:DS1307/PCF8583
Connections:
- net GND: now also DD1B1.GND
Changed lines of the file:
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@@
 <part name="XN4" library="Разъёмы штырьковые 2.54мм" deviceset="PINHD-1X13" device=""/>
 <part name="XO4" library="Разъёмы штырьковые 2.54мм" deviceset="PINHD-1X4" device=""/>
+<part name="DD1B1" library="ds1307_pcf8583" deviceset="DS1307" device="/PCF8583" value="DS1307/PCF8583"/>
+<part name="GND1" library="supply1" deviceset="GND" device=""/>
 </parts>
 <sheets>
@@
 <attribute name="VALUE" x="41.91" y="176.022" size="1.778" layer="96" rot="R180"/>
 </instance>
+<instance part="DD1B1" gate="G$1" x="-20.32" y="152.4"/>
+<instance part="GND1" gate="1" x="-33.02" y="139.7"/>
 </instances>
 <busses>
@@
 <wire x1="157.48" y1="132.08" x2="157.48" y2="129.54" width="0.1524" layer="91"/>
 </segment>
+<segment>
+<pinref part="GND1" gate="1" pin="GND"/>
+<wire x1="-33.02" y1="142.24" x2="-33.02" y2="144.78" width="0.1524" layer="91"/>
+<pinref part="DD1B1" gate="G$1" pin="GND"/>
+<wire x1="-33.02" y1="144.78" x2="-30.48" y2="144.78" width="0.1524" layer="91"/>
+</segment>
 </net>

Commit message: .
Parts:
- removed DATAIN: (no value), Разъёмы штырьковые 2.54мм:PINHD-1X3
- removed QO1, QO2: (no value), Разъёмы штырьковые 2.54мм:PINHD-1X1
- added JP2: (no value), Разъёмы штырьковые 2.54мм:PINHD-1X5
Connections:
- net RCLOCK: now also JP2.3; no longer DATAIN.1
- net RLATCH: now also JP2.2; no longer DATAIN.2
- net SER0: now also JP2.1; no longer DATAIN.3
- net SER1: now also JP2.4; no longer QO1.1
- net SER2: now also JP2.5; no longer QO2.1
Other:
- note added: "Q1 Q2"
